Commit message: lbr_iiwa_description: first kinda working version

File: lbr_iiwa_description/urdf/lbr_iiwa.urdf.xacro (robot description, xacro)
@@ -1,5 +1,5 @@
 <?xml version="1.0"?>
-<robot name="lwr">
-  <xacro:include filename="$(find lbr_iiwa_description)/urdf/lbr_iiwa.xacro"/>
+<robot name="lbr_iiwa" xmlns:xacro="http://www.ros.org/wiki/xacro">
+<xacro:include filename="$(find lbr_iiwa_description)/urdf/lbr_iiwa.xacro"/>
   <link name="world_link">
     <inertial>
@@ -16,5 +16,4 @@
       </geometry>
     </visual>
->
     <collision>
       <origin xyz="0 0 0.50" rpy="0 0 0"/>
@@ -22,8 +21,8 @@
         <box size="1 1 1.0"/>
       </geometry>
-    </collision> -->
+    </collision>
   </link>
   <lbr_iiwa parent="world" name="lbr_iiwa" right="1">
     <origin xyz="0 0 1.1" rpy="0 0 0"/>
-  </lwr_arm>
+  </lbr_iiwa>
 </robot>

File: lbr_iiwa_description/urdf/lbr_iiwa.xacro (robot description, xacro)
@@ -46,291 +46,4 @@
       </collision>
     </link>
-<!-- joint between arm_0_link and arm_1_link -->
-    <joint name="${name}_1_joint" type="revolute">
-		<parent link="${name}_0_link"/>
-		<child link="${name}_1_link"/>
-      <origin xyz="0 0 0.11" rpy="0 0 0"/>
-      <axis xyz="0 0 1"/>
-      <limit lower="${-170 * M_PI / 180}" upper="${170 * M_PI / 180}"
-             effort="204" velocity="${velocity_scale_factor * 110 * M_PI / 180}" />
-   <!--   <safety_controller soft_lower_limit="${-168 * M_PI / 180}"
-                         soft_upper_limit="${168 * M_PI / 180}"
-                         k_position="${safety_controller_k_pos}"
-                         k_velocity="${safety_controller_k_vel}"/> -->
-      <dynamics damping="${joint_damping}"/>
-    </joint>
-    <link name="${name}_1_link">
-      <inertial>
-        <mass value="${link_mass}"/>
-        <origin rpy="0 0 0" xyz="0 0 0.130"/>
-        <cuboid_inertia_def length="0.12" width="0.06" height="0.260"
-                            mass="${link_mass}"/>
-      </inertial>
-      <visual>
-        <origin xyz="0 0 0" rpy="0 0 ${M_PI}"/>
-        <geometry>
-          <mesh filename="package://lbr_iiwa_description/meshes/link_1.stl"/>
-        </geometry>
-        <material name="Orange"/>
-      </visual>
-		<collision>
-        <origin xyz="0 0 0" rpy="0 0 ${M_PI}"/>
-        <geometry>
-          <mesh filename="package://lbr_iiwa_description/meshes/link_1.stl"/>
-        </geometry>
-        <material name="Orange"/>
-		</collision>
-    </link>
-  <!--  <transmission name="${name}_arm_0_trans" type="pr2_mechanism_model/SimpleTransmission">
-      <actuator name="${name}_arm_0_motor"/>
-      <joint name="${name}_arm_0_joint"/>
-      <mechanicalReduction>1.0</mechanicalReduction>
-    </transmission> -->
-        <!-- joint between arm_1_link and arm_2_link -->
-    <joint name="${name}_2_joint" type="revolute">
-		<parent link="${name}_1_link"/>
-		<child link="${name}_2_link"/>
-      <origin xyz="0 0 0.20" rpy="0 0 0"/>
-      <axis xyz="0 -1 0"/>
-      <limit lower="${-120 * M_PI / 180}" upper="${120 * M_PI / 180}"
-          effort="306" velocity="${arm_velocity_scale_factor * 110 * M_PI / 180}" />
-     <!-- <safety_controller soft_lower_limit="${-118 * M_PI / 180}"
-                         soft_upper_limit="${118 * M_PI / 180}"
-                         k_position="${safety_controller_k_pos}"
-                         k_velocity="${safety_controller_k_vel}"/> -->
-      <dynamics damping="${joint_damping}"/>
-    </joint>
-    <link name="${name}_2_link">
-      <inertial>
-        <mass value="${link_mass}"/>
-        <origin rpy="0 0 0" xyz="0 0.06 ${0.130 - 0.06}"/>
-        <cuboid_inertia length="0.12" width="0.06" height="0.260"
-                            mass="${link_mass}"/>
-      </inertial>
-      <visual>
-        <origin xyz="0 0 0.2" rpy="${M_PI} 0 ${M_PI}"/>
-        <geometry>
-          <mesh filename="package://lbr_iiwa_description/meshes/link_2.stl"/>
-        </geometry>
-        <material name="Orange"/>
-      </visual>
-      <collision>
-        <origin xyz="0 0 0.2" rpy="${M_PI} 0 ${M_PI}"/>
-        <geometry>
-          <mesh filename="package://lbr_iiwa_description/meshes/link_2.stl"/>
-        </geometry>
-        <material name="Orange"/>
-      </collision>
-    </link>
-  <!--  <transmission name="${name}_arm_1_trans" type="pr2_mechanism_model/SimpleTransmission">
-      <actuator name="${name}_arm_1_motor"/>
-      <joint name="${name}_arm_1_joint"/>
-      <mechanicalReduction>1.0</mechanicalReduction>
-    </transmission> -->
-  <!-- joint between arm_2_link and arm_3_link -->
-    <joint name="${name}_3_joint" type="revolute">
-		<parent link="${name}_2_link"/>
-		<child link="${name}_3_link"/>
-      <origin xyz="0 0 0.20" rpy="0 0 0"/>
-      <axis xyz="0 0 1"/>
-      <limit lower="${-170 * M_PI / 180}" upper="${170 * M_PI / 180}"
-             effort="204" velocity="${arm_velocity_scale_factor * 130 * M_PI / 180}" />
-      <!--<safety_controller soft_lower_limit="${-168 * M_PI / 180}"
-                         soft_upper_limit="${168 * M_PI / 180}"
-                         k_position="${safety_controller_k_pos}"
-                         k_velocity="${safety_controller_k_vel}"/> -->
-      <dynamics damping="${joint_damping}"/>
-    </joint>
-    <link name="${name}_3_link">
-      <inertial>
-        <mass value="${link_mass}"/>
-        <origin rpy="0 0 0" xyz="0 0.06 0.130"/>
-        <cuboid_inertia_def length="0.12" width="0.06" height="0.260"
-                            mass="${link_mass}"/>
-      </inertial>
-      <visual>
-        <origin xyz="0 0 0" rpy="0 0 0"/>
-        <geometry>
-          <mesh filename="package://lbr_iiwa_description/meshes/link_3.stl"/>
-        </geometry>
-        <material name="Orange"/>
-      </visual>
-      <collision>
-        <origin xyz="0 0 0" rpy="0 0 0"/>
-        <geometry>
-          <mesh filename="package://lbr_iiwa_description/meshes/link_3.stl"/>
-        </geometry>
-        <material name="Orange"/>
-      </collision>
-    </link>
-  <!--  <transmission name="${name}_arm_2_trans" type="pr2_mechanism_model/SimpleTransmission">
-      <actuator name="${name}_arm_2_motor"/>
-      <joint name="${name}_arm_2_joint"/>
-      <mechanicalReduction>1.0</mechanicalReduction>
-    </transmission> -->
-        <!-- joint between arm_3_link and arm_4_link -->
-    <joint name="${name}_4_joint" type="revolute">
-		<parent link="${name}_3_link"/>
-		<child link="${name}_4_link"/>
-      <origin xyz="0 0 0.20" rpy="0 0 0"/>
-      <axis xyz="0 1 0"/>
-      <limit lower="${-120 * M_PI / 180}" upper="${120 * M_PI / 180}"
-             effort="306" velocity="${arm_velocity_scale_factor * 130 * M_PI / 180}" />
-     <!-- <safety_controller soft_lower_limit="${-118 * M_PI / 180}"
-                         soft_upper_limit="${118 * M_PI / 180}"
-                         k_position="${safety_controller_k_pos}"
-                         k_velocity="${safety_controller_k_vel}"/>-->
-      <dynamics damping="${joint_damping}"/>
-    </joint>
-    <link name="${name}_4_link">
-      <inertial>
-        <mass value="${link_mass}"/>
-        <origin rpy="0 0 0" xyz="0 -0.06 ${0.130 - 0.06}"/>
-        <cuboid_inertia length="0.12" width="0.06" height="0.2600"
-                            mass="${link_mass}"/>
-      </inertial>
-      <visual>
-        <origin xyz="0 0 0.2" rpy="0 ${M_PI} ${M_PI}"/>
-        <geometry>
-          <mesh filename="package://lbr_iiwa_description/meshes/link_4.stl"/>
-        </geometry>
-        <material name="Orange"/>
-      </visual>
-      <collision>
-       <origin xyz="0 0 0.2" rpy="0 ${M_PI} ${M_PI}"/>
-        <geometry>
-          <mesh filename="package://lbr_iiwa_description/meshes/link_4.stl"/>
-        </geometry>
-        <material name="Orange"/>
-      </collision>
-    </link>
-  <!--  <transmission name="${name}_arm_3_trans" type="pr2_mechanism_model/SimpleTransmission">
-      <actuator name="${name}_arm_3_motor"/>
-      <joint name="${name}_arm_3_joint"/>
-      <mechanicalReduction>1.0</mechanicalReduction>
-    </transmission> -->
-        <!-- joint between arm_4_link and arm_5_link -->
-    <joint name="${name}_5_joint" type="revolute">
-		<parent link="${name}_4_link"/>
-		<child link="${name}_5_link"/>
-      <origin xyz="0 0 0.20" rpy="0 0 0"/>
-      <axis xyz="0 0 1"/>
-      <limit lower="${-170 * M_PI / 180}" upper="${170 * M_PI / 180}"
-             effort="204" velocity="${arm_velocity_scale_factor * 130 * M_PI / 180}" />
-     <!-- <safety_controller soft_lower_limit="${-168 * M_PI / 180}"
-                         soft_upper_limit="${168 * M_PI / 180}"
-                         k_position="${safety_controller_k_pos}"
-                         k_velocity="${safety_controller_k_vel}"/> -->
-      <dynamics damping="${joint_damping}"/>
-    </joint>
-    <link name="${name}_5_link">
-      <inertial>
-        <mass value="${link_mass}"/>
-        <origin rpy="0 0 0" xyz="0 0 0.124"/>
-        <cuboid_inertia length="0.12" width="0.06" height="0.248"
-                            mass="${link_mass}"/>
-      </inertial>
-      <visual>
-        <origin xyz="0 0 0" rpy="0 0 ${M_PI}"/>
-        <geometry>
-          <mesh filename="package://lbr_iiwa_description/meshes/link_5.stl"/>
-        </geometry>
-        <material name="Orange"/>
-      </visual>
-      <collision>
-        <origin xyz="0 0 0" rpy="0 0 ${M_PI}"/>
-        <geometry>
-          <mesh filename="package://lbr_iiwa_description/meshes/link_5.stl"/>
-        </geometry>
-        <material name="Orange"/>
-      </collision>
-    </link>
-  <!-- <transmission name="${name}_arm_4_trans" type="pr2_mechanism_model/SimpleTransmission">
-      <actuator name="${name}_arm_4_motor"/>
-      <joint name="${name}_arm_4_joint"/>
-      <mechanicalReduction>1.0</mechanicalReduction>
-    </transmission> -->
-  <!-- joint between arm_5_link and arm_6_link -->
-    <joint name="${name}_6_joint" type="revolute">
-  		<parent link="${name}_5_link"/>
-		<child link="${name}_6_link"/>
-      <origin xyz="0 0 0.19" rpy="0 0 0"/>
-      <axis xyz="0 -1 0"/>
-      <limit lower="${-120 * M_PI / 180}" upper="${120 * M_PI / 180}"
-             effort="306" velocity="${arm_velocity_scale_factor * 180 * M_PI / 180}" />
-    <!--  <safety_controller soft_lower_limit="${-118 * M_PI / 180}"
-                         soft_upper_limit="${118 * M_PI / 180}"
-                         k_position="${safety_controller_k_pos}"
-                         k_velocity="${safety_controller_k_vel}"/> -->
-      <dynamics damping="${joint_damping}"/>
-    </joint>
-    <link name="${name}_6_link">
-      <inertial>
-        <mass value="${ball_link_mass}"/>
-        <origin rpy="0 0 0" xyz="0 0 0.0625"/>
-        <cuboid_inertia length="0.125" width="0.125" height="0.125"
-                            mass="${ball_link_mass}"/>
-      </inertial>
-      <visual>
-        <origin xyz="0 0 0" rpy="0 0 ${M_PI}"/>
-        <geometry>
-          <mesh filename="package://lbr_iiwa_description/meshes/link_6.stl"/>
-        </geometry>
-        <material name="Orange"/>
-      </visual>
-      <collision>
-       <origin xyz="0 0 0" rpy="0 0 ${M_PI}"/>
-        <geometry>
-          <mesh filename="package://lbr_iiwa_description/meshes/link_6.stl"/>
-        </geometry>
-        <material name="Orange"/>
-      </collision>
-    </link>
-  <!--  <transmission name="${name}_arm_5_trans" type="pr2_mechanism_model/SimpleTransmission">
-      <actuator name="${name}_arm_5_motor"/>
-      <joint name="${name}_arm_5_joint"/>
-      <mechanicalReduction>1.0</mechanicalReduction>
-    </transmission> -->
-<!-- joint between arm_6_link and arm_7_link -->
-    <joint name="${name}_7_joint" type="revolute">
-		<parent link="${name}_6_link"/>
-		<child link="${name}_7_link"/>
-      <origin xyz="0 0 0.078" rpy="0 0 0"/>
-      <axis xyz="0 0 1"/>
-      <limit lower="${-170 * M_PI / 180}" upper="${170 * M_PI / 180}"
-             effort="204" velocity="${arm_velocity_scale_factor * 180 * M_PI / 180}" />
-      <!-- <safety_controller soft_lower_limit="${-168 * M_PI / 180}"
-                         soft_upper_limit="${168 * M_PI / 180}"
-                         k_position="${safety_controller_k_pos}"
-                         k_velocity="${safety_controller_k_vel}"/> -->
-      <dynamics damping="${joint_damping}"/>
-    </joint>
-    <link name="${name}_7_link">
-      <inertial>
-        <mass value="${end_link_mass}"/>
-        <origin xyz="0 0 0"/>
-        <cuboid_inertia_def length="1" width="1" height="1"
-                            mass="${end_link_mass}"/>
-      </inertial>
-      <visual>
-        <origin xyz="0 0 0" rpy="0 0 ${right * -1/4 * M_PI  +  M_PI}"/>
-        <geometry>
-          <mesh filename="package://lbr_iiwa_description/meshes/link_7.stl"/>
-        </geometry>
-        <material name="Grey"/>
-      </visual>
-      <collision>
-        <origin xyz="0 0 0" rpy="0 0 ${right * -1/4 * M_PI  +  M_PI}"/>
-        <geometry>
-          <mesh filename="package://lbr_iiwa_description/meshes/link_7.stl"/>
-        </geometry>
-        <material name="Grey"/>
-      </collision>
-    </link>
-  <!--  <transmission name="${name}_arm_6_trans" type="pr2_mechanism_model/SimpleTransmission">
-      <actuator name="${name}_arm_6_motor"/>
-      <joint name="${name}_arm_6_joint"/>
-      <mechanicalReduction>1.0</mechanicalReduction>
-    </transmission> -->
   </xacro:macro>
 </robot>

Commit message: modified urdf.xacro

File: lbr_iiwa_description/urdf/lbr_iiwa.urdf.xacro (robot description, xacro)
@@ -2,27 +2,9 @@
 <robot name="lbr_iiwa" xmlns:xacro="http://www.ros.org/wiki/xacro">
 <xacro:include filename="$(find lbr_iiwa_description)/urdf/lbr_iiwa.xacro"/>
-  <link name="world_link">
-    <inertial>
-      <mass value="50.0"/>
-      <com xyz="0 0 0"/>
-      <inertia  ixx="0.01" ixy="0.00"  ixz="0.00"
-                iyy="0.01" iyz="0.00"
-                izz="0.01" />
-    </inertial>
-    <visual>
-      <origin xyz="0 0 0.50" rpy="0 0 0"/>
-      <geometry>
-        <box size="1 1 1.0"/>
-      </geometry>
-    </visual>
-    <collision>
-      <origin xyz="0 0 0.50" rpy="0 0 0"/>
-      <geometry>
-        <box size="1 1 1.0"/>
-      </geometry>
-    </collision>
-  </link>
-  <lbr_iiwa parent="world" name="lbr_iiwa" right="1">
-    <origin xyz="0 0 1.1" rpy="0 0 0"/>
-  </lbr_iiwa>
+  <!-- base link-->
+  <link name="base_link"/>
+  <!--lbr-->
+  <xacro:lbr_iiwa name="arm" parent="base_link">
+    <origin xyz="0 0 0.01" rpy="0 0 0" />
+  </xacro:lbr_iiwa>
 </robot>

Commit message: lbr_iiwa_description: updated meshes

File: lbr_iiwa_description/urdf/lbr_iiwa.urdf.xacro (robot description, xacro)
@@ -1,10 +1,38 @@
 <?xml version="1.0"?>
 <robot name="lbr_iiwa" xmlns:xacro="http://www.ros.org/wiki/xacro">
-<xacro:include filename="$(find lbr_iiwa_description)/urdf/lbr_iiwa.xacro"/>
-  <!-- base link-->
-  <link name="base_link"/>
+  <xacro:include filename="$(find lbr_iiwa_description)/urdf/lbr_iiwa.xacro"/>
+  <!--  <joint name="fixed" type="fixed">
+       <parent link="world"/>
+       <child link="arm_link_0"/>
+       </joint> -->
+  <!-- Define a base link properly -->
+  <!--  <link name="base_link">
+       <collision>
+       <origin xyz="0 0 0.5" rpy="0 0 0"/>
+       <geometry>
+       <box size="1 1 1"/>
+       </geometry>
+       </collision>
+<visual>
+<origin xyz="0 0 0.5" rpy="0 0 0"/>
+<geometry>
+<box size="1 1 1"/>
+</geometry>
+<material name="orange"/>
+</visual>
+<inertial>
+<origin xyz="0 0 1" rpy="0 0 0"/>
+<mass value="1"/>
+<inertia
+ixx="1" ixy="0.0" ixz="0.0"
+iyy="1" iyz="0.0"
+izz="1"/>
+</inertial>
+</link> -->
+  <!-- Fix to world just for testing -->
+  <link name="world"/>
   <!--lbr-->
-  <xacro:lbr_iiwa name="arm" parent="base_link">
-    <origin xyz="0 0 0.01" rpy="0 0 0" />
+  <xacro:lbr_iiwa name="arm" right="1" parent="world">
+    <origin xyz="0 0 0.0" rpy="0 0 0" />
   </xacro:lbr_iiwa>
 </robot>

File: lbr_iiwa_description/urdf/lbr_iiwa.xacro (robot description, xacro)
@@ -2,5 +2,5 @@
 <robot name="lbr_iiwa" xmlns:xacro="http://www.ros.org/wiki/xacro">
   <!-- Import all Gazebo-customization elements, including Gazebo colors -->
-  <xacro:include filename="$(find lbr_iiwa_description)/urdf/lbr_iiwa.gazebo" />
+  <xacro:include filename="$(find lbr_iiwa_description)/urdf/lbr_iiwa.gazebo.xacro" />
   <!-- Import Rviz colors -->
   <xacro:include filename="$(find lbr_iiwa_description)/urdf/materials.xacro" />
@@ -8,8 +8,4 @@
   <xacro:include filename="$(find lbr_iiwa_description)/urdf/utilities.xacro"/>
   <!-- some constants -->
-  <xacro:property name="base_mass" value="2.0"/>
-  <xacro:property name="link_mass" value="2.0"/>
-  <xacro:property name="ball_link_mass" value="2.0"/>
-  <xacro:property name="end_link_mass" value="2.0"/>
   <xacro:property name="safety_controller_k_pos" value="100" />
   <xacro:property name="safety_controller_k_vel" value="2" />
@@ -18,16 +14,15 @@
   <!-- right is either 1 (for right arm) or -1 (for left arm) -->
   <xacro:macro name="lbr_iiwa" params="parent name right *origin">
-    <!--joint between {parent} and arm_0_link-->
-    <joint name="${parent}_base_joint" type="fixed">
+    <!--joint between {parent} and link_0-->
+    <joint name="${parent}_joint" type="fixed">
       <insert_block name="origin"/>
       <parent link="${parent}"/>
-      <child link="${name}_0_link"/>
+      <child link="${name}_link_0"/>
     </joint>
-    <link name="${name}_0_link">
+    <link name="${name}_link_0">
       <inertial>
-        <mass value="${base_mass}"/>
-        <origin xyz="0 0 0.055" rpy="0 0 0"/>
-        <cylinder_inertia_def radius="0.06" length="0.11"
-                              mass="${base_mass}"/>
+        <origin xyz="0 0 0.07" rpy="0 0 0"/>
+        <mass value="5"/>
+        <inertia ixx="0.05"  ixy="0"  ixz="0" iyy="0.06" iyz="0" izz="0.03" />
       </inertial>
       <visual>
@@ -36,14 +31,96 @@
           <mesh filename="package://lbr_iiwa_description/meshes/link_0.stl"/>
         </geometry>
-        <material name="Black"/>
+        <material name="Grey"/>
       </visual>
       <collision>
-           <origin xyz="0 0 0" rpy="0 0 0"/>
+        <origin xyz="0 0 0" rpy="0 0 0"/>
         <geometry>
           <mesh filename="package://lbr_iiwa_description/meshes/link_0.stl"/>
         </geometry>
-        <material name="Black"/>
+        <material name="Grey"/>
       </collision>
     </link>
+    <!-- joint between link_0 and link_1 -->
+    <joint name="${name}_joint_1" type="revolute">
+      <parent link="${name}_link_0"/>
+      <child link="${name}_link_1"/>
+      <origin xyz="0 0 0.1575" rpy="0 0 0"/>
+      <axis xyz="0 0 1"/>
+      <limit lower="${-170 * PI / 180}" upper="${170 * PI / 180}"
+             effort="204" velocity="${velocity_scale_factor * 110 * PI / 180}" />
+      <!--   <safety_controller soft_lower_limit="${-168 * M_PI / 180}"
+           soft_upper_limit="${168 * M_PI / 180}"
+           k_position="${safety_controller_k_pos}"
+           k_velocity="${safety_controller_k_vel}"/> -->
+      <dynamics damping="${joint_damping}"/>
+    </joint>
+    <link name="${name}_link_1">
+      <inertial>
+        <origin xyz="0 0.03 0.12" rpy="0 0 0"/>
+        <mass value="4"/>
+        <inertia ixx="0.1"  ixy="0"  ixz="0" iyy="0.09" iyz="0" izz="0.02" />
+      </inertial>
+      <visual>
+        <origin xyz="0 0 0" rpy="0 0 0"/>
+        <geometry>
+          <mesh filename="package://lbr_iiwa_description/meshes/link_1.stl"/>
+        </geometry>
+        <material name="Orange"/>
+      </visual>
+      <collision>
+        <origin xyz="0 0 0" rpy="0 0 0"/>
+        <geometry>
+          <mesh filename="package://lbr_iiwa_description/meshes/link_1.stl"/>
+        </geometry>
+        <material name="Orange"/>
+      </collision>
+    </link>
+    <!--  <transmission name="${name}_arm_0_trans" type="pr2_mechanism_model/SimpleTransmission">
+	 <actuator name="${name}_arm_0_motor"/>
+	 <joint name="${name}_arm_0_joint"/>
+	 <mechanicalReduction>1.0</mechanicalReduction>
+	 </transmission> -->
+    <!-- joint between link_1 and link_2 -->
+    <joint name="${name}_joint_2" type="revolute">
+      <parent link="${name}_link_1"/>
+      <child link="${name}_link_2"/>
+      <origin xyz="0 0 0.20" rpy="0 0 0"/>
+      <axis xyz="0 0 1"/>
+      <limit lower="${-120 * PI / 180}" upper="${120 * PI / 180}"
+             effort="306" velocity="${velocity_scale_factor * 110 * PI / 180}" />
+      <!-- <safety_controller soft_lower_limit="${-118 * PI / 180}"
+           soft_upper_limit="${118 * PI / 180}"
+           k_position="${safety_controller_k_pos}"
+           k_velocity="${safety_controller_k_vel}"/> -->
+      <dynamics damping="${joint_damping}"/>
+    </joint>
+    <link name="${name}_link_2">
+      <inertial>
+        <origin xyz="0 0.06 0.04" rpy="0 0 0"/>
+        <mass value="4"/>
+        <inertia ixx="0.05"  ixy="0"  ixz="0" iyy="0.02" iyz="0" izz="0.04" />
+      </inertial>
+      <visual>
+        <origin xyz="0 0 0" rpy="0 0 0"/>
+        <geometry>
+          <mesh filename="package://lbr_iiwa_description/meshes/link_2.stl"/>
+        </geometry>
+        <material name="Orange"/>
+      </visual>
+      <collision>
+        <origin xyz="0 0 0" rpy="0 0 0"/>
+        <geometry>
+          <mesh filename="package://lbr_iiwa_description/meshes/link_2.stl"/>
+        </geometry>
+        <material name="Orange"/>
+      </collision>
+    </link>
+    <!--  <transmission name="${name}_arm_1_trans" type="pr2_mechanism_model/SimpleTransmission">
+	 <actuator name="${name}_arm_1_motor"/>
+	 <joint name="${name}_arm_1_joint"/>
+	 <mechanicalReduction>1.0</mechanicalReduction>
+	 </transmission> -->
+    <!--Extensions -->
+    <xacro:lbr_iiwa_gazebo name="${name}" />
   </xacro:macro>
 </robot>

File: lbr_iiwa_description/urdf/utilities.xacro (robot description, xacro)
@@ -5,21 +5,15 @@
   <!--Cuboid-->
   <xacro:macro name="cuboid_inertia" params="width height length mass">
-    <inertial>
-    <mass value="${mass}" />
     <inertia ixx="${mass * (height * height + length * length) / 12)}"
              iyy="${mass * (width * width + length * length) / 12)}"
              izz="${mass * (width * width + height * height) / 12)}"
              ixy="0" iyz="0" ixz="0"/>
-    </inertial>
   </xacro:macro>
   <!--Cylinder: length is along the y-axis! -->
   <xacro:macro name="cylinder_inertia" params="radius length mass">
-  <inertial>
-    <mass value="${mass}" />
     <inertia ixx="${mass * (3 * radius * radius + length * length) / 12)}"
              iyy="${mass * radius* radius / 2)}"
              izz="${mass * (3 * radius * radius + length * length) / 12)}"
              ixy="0" iyz="0" ixz="0"/>
-    </inertial>
   </xacro:macro>
 </robot>
