Commit message: added lbr_iiwa_control package

File: lbr_iiwa_description/urdf/lbr_iiwa.gazebo.xacro (robot description, xacro)
@@ -2,4 +2,10 @@
 <robot name="lbr_iiwa" xmlns:xacro="http://www.ros.org/wiki/xacro">
   <xacro:macro name="lbr_iiwa_gazebo" params="name">
+    <!-- ros_control plugin -->
+    <gazebo>
+      <plugin name="gazebo_ros_control" filename="libgazebo_ros_control.so">
+	<robotNamespace>/lbr_iiwa</robotNamespace>
+      </plugin>
+    </gazebo>
     <!-- Link0 -->
     <gazebo reference="${name}_link_0">

File: lbr_iiwa_description/urdf/lbr_iiwa.urdf.xacro (robot description, xacro)
@@ -33,5 +33,5 @@
   <link name="world"/>
   <!--lbr-->
-  <xacro:lbr_iiwa name="arm" right="1" parent="world">
+  <xacro:lbr_iiwa name="lbr_iiwa" right="1" parent="world">
     <origin xyz="0 0 0.0" rpy="0 0 0" />
   </xacro:lbr_iiwa>

File: lbr_iiwa_description/urdf/lbr_iiwa.xacro (robot description, xacro)
@@ -8,6 +8,6 @@
   <xacro:include filename="$(find lbr_iiwa_description)/urdf/utilities.xacro"/>
   <!-- some constants -->
-  <xacro:property name="safety_controller_k_pos" value="100" />
-  <xacro:property name="safety_controller_k_vel" value="2" />
+ <!-- <xacro:property name="safety_controller_k_pos" value="100" />
+  <xacro:property name="safety_controller_k_vel" value="2" /> -->
   <xacro:property name="joint_damping" value="0.1" />
   <xacro:property name="velocity_scale_factor" value="1"/>
@@ -288,4 +288,5 @@
     <!--Extensions -->
     <xacro:lbr_iiwa_gazebo name="${name}" />
+    <xacro:lbr_iiwa_transmission name="${name}" />
   </xacro:macro>
 </robot>
