Commit message: lbr_iiwa_control: position controllers work now

File: lbr_iiwa_description/urdf/lbr_iiwa.transmission.xacro (robot description, xacro)
@@ -2,70 +2,70 @@
 <robot name="lbr_iiwa" xmlns:xacro="http://www.ros.org/wiki/xacro">
   <xacro:macro name="lbr_iiwa_transmission" params="name">
-    <transmission name="{name}_tran_1">
+    <transmission name="${name}_tran_1">
       <type>transmission_interface/SimpleTransmission</type>
-      <joint name="{name}_joint_1">
+      <joint name="${name}_joint_1">
 	<hardwareInterface>EffortJointInterface</hardwareInterface>
       </joint>
-      <actuator name="{name}_motor_1">
+      <actuator name="${name}_motor_1">
 	<hardwareInterface>EffortJointInterface</hardwareInterface>
 	<mechanicalReduction>1</mechanicalReduction>
       </actuator>
     </transmission>
-    <transmission name="{name}_tran_2">
+    <transmission name="${name}_tran_2">
       <type>transmission_interface/SimpleTransmission</type>
-      <joint name="{name}_joint_2">
+      <joint name="${name}_joint_2">
 	<hardwareInterface>EffortJointInterface</hardwareInterface>
       </joint>
-      <actuator name="{name}_motor_2">
+      <actuator name="${name}_motor_2">
 	<hardwareInterface>EffortJointInterface</hardwareInterface>
 	<mechanicalReduction>1</mechanicalReduction>
       </actuator>
     </transmission>
-    <transmission name="{name}_tran_3">
+    <transmission name="${name}_tran_3">
       <type>transmission_interface/SimpleTransmission</type>
-      <joint name="{name}_joint_3">
+      <joint name="${name}_joint_3">
 	<hardwareInterface>EffortJointInterface</hardwareInterface>
       </joint>
-      <actuator name="{name}_motor_3">
+      <actuator name="${name}_motor_3">
 	<hardwareInterface>EffortJointInterface</hardwareInterface>
 	<mechanicalReduction>1</mechanicalReduction>
       </actuator>
     </transmission>
-    <transmission name="{name}_tran_4">
+    <transmission name="${name}_tran_4">
       <type>transmission_interface/SimpleTransmission</type>
-      <joint name="{name}_joint_4">
+      <joint name="${name}_joint_4">
 	<hardwareInterface>EffortJointInterface</hardwareInterface>
       </joint>
-      <actuator name="{name}_motor_4">
+      <actuator name="${name}_motor_4">
 	<hardwareInterface>EffortJointInterface</hardwareInterface>
 	<mechanicalReduction>1</mechanicalReduction>
       </actuator>
     </transmission>
-    <transmission name="{name}_tran_5">
+    <transmission name="${name}_tran_5">
       <type>transmission_interface/SimpleTransmission</type>
-      <joint name="{name}_joint_5">
+      <joint name="${name}_joint_5">
 	<hardwareInterface>EffortJointInterface</hardwareInterface>
       </joint>
-      <actuator name="{name}_motor_5">
+      <actuator name="${name}_motor_5">
 	<hardwareInterface>EffortJointInterface</hardwareInterface>
 	<mechanicalReduction>1</mechanicalReduction>
       </actuator>
     </transmission>
-    <transmission name="{name}_tran_6">
+    <transmission name="${name}_tran_6">
       <type>transmission_interface/SimpleTransmission</type>
-      <joint name="{name}_joint_6">
+      <joint name="${name}_joint_6">
 	<hardwareInterface>EffortJointInterface</hardwareInterface>
       </joint>
-      <actuator name="{name}_motor_6">
+      <actuator name="${name}_motor_6">
 	<hardwareInterface>EffortJointInterface</hardwareInterface>
 	<mechanicalReduction>1</mechanicalReduction>
       </actuator>
     </transmission>
-    <transmission name="{name}_tran_7">
+    <transmission name="${name}_tran_7">
       <type>transmission_interface/SimpleTransmission</type>
-      <joint name="{name}_joint_7">
+      <joint name="${name}_joint_7">
 	<hardwareInterface>EffortJointInterface</hardwareInterface>
       </joint>
-      <actuator name="{name}_motor_7">
+      <actuator name="${name}_motor_7">
 	<hardwareInterface>EffortJointInterface</hardwareInterface>
 	<mechanicalReduction>1</mechanicalReduction>

File: lbr_iiwa_description/urdf/lbr_iiwa.xacro (robot description, xacro)
@@ -5,6 +5,8 @@
   <!-- Import Rviz colors -->
   <xacro:include filename="$(find lbr_iiwa_description)/urdf/materials.xacro" />
-  <!-- Import Utilities -->
-  <xacro:include filename="$(find lbr_iiwa_description)/urdf/utilities.xacro"/>
+  <!-- Import Transmissions -->
+  <xacro:include filename="$(find lbr_iiwa_description)/urdf/lbr_iiwa.transmission.xacro" />
+  <!-- Include Utilities -->
+  <xacro:include filename="$(find lbr_iiwa_description)/urdf/utilities.xacro" />
   <!-- some constants -->
  <!-- <xacro:property name="safety_controller_k_pos" value="100" />

Commit message: cleaned up the launch files

File: lbr_iiwa_description/urdf/lbr_iiwa.transmission.xacro (robot description, xacro)
@@ -1,12 +1,12 @@
 <?xml version="1.0"?>
 <robot name="lbr_iiwa" xmlns:xacro="http://www.ros.org/wiki/xacro">
-  <xacro:macro name="lbr_iiwa_transmission" params="name">
+  <xacro:macro name="lbr_iiwa_transmission" params="name hardware_interface">
     <transmission name="${name}_tran_1">
       <type>transmission_interface/SimpleTransmission</type>
       <joint name="${name}_joint_1">
-	<hardwareInterface>EffortJointInterface</hardwareInterface>
+	<hardwareInterface>${hardware_interface}</hardwareInterface>
       </joint>
       <actuator name="${name}_motor_1">
-	<hardwareInterface>EffortJointInterface</hardwareInterface>
+	<hardwareInterface>${hardware_interface}</hardwareInterface>
 	<mechanicalReduction>1</mechanicalReduction>
       </actuator>
@@ -15,8 +15,8 @@
       <type>transmission_interface/SimpleTransmission</type>
       <joint name="${name}_joint_2">
-	<hardwareInterface>EffortJointInterface</hardwareInterface>
+	<hardwareInterface>${hardware_interface}</hardwareInterface>
       </joint>
       <actuator name="${name}_motor_2">
-	<hardwareInterface>EffortJointInterface</hardwareInterface>
+	<hardwareInterface>${hardware_interface}</hardwareInterface>
 	<mechanicalReduction>1</mechanicalReduction>
       </actuator>
@@ -25,8 +25,8 @@
       <type>transmission_interface/SimpleTransmission</type>
       <joint name="${name}_joint_3">
-	<hardwareInterface>EffortJointInterface</hardwareInterface>
+	<hardwareInterface>${hardware_interface}</hardwareInterface>
       </joint>
       <actuator name="${name}_motor_3">
-	<hardwareInterface>EffortJointInterface</hardwareInterface>
+	<hardwareInterface>${hardware_interface}</hardwareInterface>
 	<mechanicalReduction>1</mechanicalReduction>
       </actuator>
@@ -35,8 +35,8 @@
       <type>transmission_interface/SimpleTransmission</type>
       <joint name="${name}_joint_4">
-	<hardwareInterface>EffortJointInterface</hardwareInterface>
+	<hardwareInterface>${hardware_interface}</hardwareInterface>
       </joint>
       <actuator name="${name}_motor_4">
-	<hardwareInterface>EffortJointInterface</hardwareInterface>
+	<hardwareInterface>${hardware_interface}</hardwareInterface>
 	<mechanicalReduction>1</mechanicalReduction>
       </actuator>
@@ -45,8 +45,8 @@
       <type>transmission_interface/SimpleTransmission</type>
       <joint name="${name}_joint_5">
-	<hardwareInterface>EffortJointInterface</hardwareInterface>
+	<hardwareInterface>${hardware_interface}</hardwareInterface>
       </joint>
       <actuator name="${name}_motor_5">
-	<hardwareInterface>EffortJointInterface</hardwareInterface>
+	<hardwareInterface>${hardware_interface}</hardwareInterface>
 	<mechanicalReduction>1</mechanicalReduction>
       </actuator>
@@ -55,8 +55,8 @@
       <type>transmission_interface/SimpleTransmission</type>
       <joint name="${name}_joint_6">
-	<hardwareInterface>EffortJointInterface</hardwareInterface>
+	<hardwareInterface>${hardware_interface}</hardwareInterface>
       </joint>
       <actuator name="${name}_motor_6">
-	<hardwareInterface>EffortJointInterface</hardwareInterface>
+	<hardwareInterface>${hardware_interface}</hardwareInterface>
 	<mechanicalReduction>1</mechanicalReduction>
       </actuator>
@@ -65,8 +65,8 @@
       <type>transmission_interface/SimpleTransmission</type>
       <joint name="${name}_joint_7">
-	<hardwareInterface>EffortJointInterface</hardwareInterface>
+	<hardwareInterface>${hardware_interface}</hardwareInterface>
       </joint>
       <actuator name="${name}_motor_7">
-	<hardwareInterface>EffortJointInterface</hardwareInterface>
+	<hardwareInterface>${hardware_interface}</hardwareInterface>
 	<mechanicalReduction>1</mechanicalReduction>
       </actuator>

File: lbr_iiwa_description/urdf/lbr_iiwa.urdf.xacro (robot description, xacro)
@@ -2,36 +2,8 @@
 <robot name="lbr_iiwa" xmlns:xacro="http://www.ros.org/wiki/xacro">
   <xacro:include filename="$(find lbr_iiwa_description)/urdf/lbr_iiwa.xacro"/>
-  <!--  <joint name="fixed" type="fixed">
-       <parent link="world"/>
-       <child link="arm_link_0"/>
-       </joint> -->
-  <!-- Define a base link properly -->
-  <!--  <link name="base_link">
-       <collision>
-       <origin xyz="0 0 0.5" rpy="0 0 0"/>
-       <geometry>
-       <box size="1 1 1"/>
-       </geometry>
-       </collision>
-<visual>
-<origin xyz="0 0 0.5" rpy="0 0 0"/>
-<geometry>
-<box size="1 1 1"/>
-</geometry>
-<material name="orange"/>
-</visual>
-<inertial>
-<origin xyz="0 0 1" rpy="0 0 0"/>
-<mass value="1"/>
-<inertia
-ixx="1" ixy="0.0" ixz="0.0"
-iyy="1" iyz="0.0"
-izz="1"/>
-</inertial>
-</link> -->
   <!-- Fix to world just for testing -->
   <link name="world"/>
   <!--lbr-->
-  <xacro:lbr_iiwa name="lbr_iiwa" right="1" parent="world">
+  <xacro:lbr_iiwa name="lbr_iiwa" hardware_interface="$(arg prefix)" parent="world">
     <origin xyz="0 0 0.0" rpy="0 0 0" />
   </xacro:lbr_iiwa>

File: lbr_iiwa_description/urdf/lbr_iiwa.xacro (robot description, xacro)
@@ -15,6 +15,5 @@
   <xacro:property name="max_effort" value="300"/>
   <xacro:property name="max_velocity" value="10"/>
-  <!-- right is either 1 (for right arm) or -1 (for left arm) -->
-  <xacro:macro name="lbr_iiwa" params="parent name right *origin">
+  <xacro:macro name="lbr_iiwa" params="parent name hardware_interface *origin">
     <!--joint between {parent} and link_0-->
     <joint name="${parent}_joint" type="fixed">
@@ -291,5 +290,5 @@
     <!--Extensions -->
     <xacro:lbr_iiwa_gazebo name="${name}" />
-    <xacro:lbr_iiwa_transmission name="${name}" />
+    <xacro:lbr_iiwa_transmission name="${name}" hardware_interface="${hardware_interface}"/>
   </xacro:macro>
 </robot>
