Commit message: first working version of the urdf (party)

File: lbr_iiwa_description/urdf/lbr_iiwa.xacro (robot description, xacro)
@@ -22,5 +22,5 @@
     <link name="${name}_link_0">
       <inertial>
-        <origin xyz="0 0 0.07" rpy="0 0 0"/>
+        <origin xyz="-0.1 0 0.07" rpy="0 0 0"/>
         <mass value="5"/>
         <inertia ixx="0.05"  ixy="0"  ixz="0" iyy="0.06" iyz="0" izz="0.03" />
@@ -57,5 +57,5 @@
     <link name="${name}_link_1">
       <inertial>
-        <origin xyz="0 0.03 0.12" rpy="0 0 0"/>
+        <origin xyz="0 -0.03 0.12" rpy="0 0 0"/>
         <mass value="4"/>
         <inertia ixx="0.1"  ixy="0"  ixz="0" iyy="0.09" iyz="0" izz="0.02" />
@@ -76,15 +76,10 @@
       </collision>
     </link>
-    <!--  <transmission name="${name}_arm_0_trans" type="pr2_mechanism_model/SimpleTransmission">
-	 <actuator name="${name}_arm_0_motor"/>
-	 <joint name="${name}_arm_0_joint"/>
-	 <mechanicalReduction>1.0</mechanicalReduction>
-	 </transmission> -->
     <!-- joint between link_1 and link_2 -->
     <joint name="${name}_joint_2" type="revolute">
       <parent link="${name}_link_1"/>
       <child link="${name}_link_2"/>
-      <origin xyz="0 0 0.20" rpy="0 0 0"/>
-      <axis xyz="0 0 1"/>
+      <origin xyz="0 0 0.2025" rpy="0 0 0"/>
+      <axis xyz="0 1 0"/>
       <limit lower="${-120 * PI / 180}" upper="${120 * PI / 180}"
              effort="306" velocity="${velocity_scale_factor * 110 * PI / 180}" />
@@ -97,7 +92,7 @@
     <link name="${name}_link_2">
       <inertial>
-        <origin xyz="0 0.06 0.04" rpy="0 0 0"/>
+        <origin xyz="0 0.04 0.06" rpy="0 0 0"/>
         <mass value="4"/>
-        <inertia ixx="0.05"  ixy="0"  ixz="0" iyy="0.02" iyz="0" izz="0.04" />
+        <inertia ixx="0.05"  ixy="0"  ixz="0" iyy="0.04" iyz="0" izz="0.02" />
       </inertial>
       <visual>
@@ -116,9 +111,179 @@
       </collision>
     </link>
-    <!--  <transmission name="${name}_arm_1_trans" type="pr2_mechanism_model/SimpleTransmission">
-	 <actuator name="${name}_arm_1_motor"/>
-	 <joint name="${name}_arm_1_joint"/>
-	 <mechanicalReduction>1.0</mechanicalReduction>
-	 </transmission> -->
+    <!-- joint between link_2 and link_3 -->
+    <joint name="${name}_joint_3" type="revolute">
+      <parent link="${name}_link_2"/>
+      <child link="${name}_link_3"/>
+      <origin xyz="0 0 0.2045" rpy="0 0 0"/>
+      <axis xyz="0 0 1"/>
+      <limit lower="${-170 * PI / 180}" upper="${170 * PI / 180}"
+             effort="306" velocity="${velocity_scale_factor * 110 * PI / 180}" />
+      <!-- <safety_controller soft_lower_limit="${-118 * PI / 180}"
+           soft_upper_limit="${118 * PI / 180}"
+           k_position="${safety_controller_k_pos}"
+           k_velocity="${safety_controller_k_vel}"/> -->
+      <dynamics damping="${joint_damping}"/>
+    </joint>
+    <link name="${name}_link_3">
+      <inertial>
+        <origin xyz="0 0.03 0.13" rpy="0 0 0"/>
+        <mass value="3"/>
+        <inertia ixx="0.08"  ixy="0"  ixz="0" iyy="0.07" iyz="0" izz="0.01" />
+      </inertial>
+      <visual>
+        <origin xyz="0 0 0" rpy="0 0 0"/>
+        <geometry>
+          <mesh filename="package://lbr_iiwa_description/meshes/link_3.stl"/>
+        </geometry>
+        <material name="Orange"/>
+      </visual>
+      <collision>
+        <origin xyz="0 0 0" rpy="0 0 0"/>
+        <geometry>
+          <mesh filename="package://lbr_iiwa_description/meshes/link_3.stl"/>
+        </geometry>
+        <material name="Orange"/>
+      </collision>
+    </link>
+   <!-- joint between link_3 and link_4 -->
+    <joint name="${name}_joint_4" type="revolute">
+      <parent link="${name}_link_3"/>
+      <child link="${name}_link_4"/>
+      <origin xyz="0 0 0.2155" rpy="0 0 0"/>
+      <axis xyz="0 1 0"/>
+      <limit lower="${-120 * PI / 180}" upper="${120 * PI / 180}"
+             effort="306" velocity="${velocity_scale_factor * 110 * PI / 180}" />
+      <!-- <safety_controller soft_lower_limit="${-118 * PI / 180}"
+           soft_upper_limit="${118 * PI / 180}"
+           k_position="${safety_controller_k_pos}"
+           k_velocity="${safety_controller_k_vel}"/> -->
+      <dynamics damping="${joint_damping}"/>
+    </joint>
+    <link name="${name}_link_4">
+      <inertial>
+        <origin xyz="0 -0.03 0.07" rpy="0 0 0"/>
+        <mass value="2.5"/>
+        <inertia ixx="0.03"  ixy="0"  ixz="0" iyy="0.03" iyz="0" izz="0.01" />
+      </inertial>
+      <visual>
+        <origin xyz="0 0 0" rpy="0 0 0"/>
+        <geometry>
+          <mesh filename="package://lbr_iiwa_description/meshes/link_4.stl"/>
+        </geometry>
+        <material name="Orange"/>
+      </visual>
+      <collision>
+        <origin xyz="0 0 0" rpy="0 0 0"/>
+        <geometry>
+          <mesh filename="package://lbr_iiwa_description/meshes/link_4.stl"/>
+        </geometry>
+        <material name="Orange"/>
+      </collision>
+    </link>
+    <!-- joint between link_4 and link_5 -->
+    <joint name="${name}_joint_5" type="revolute">
+      <parent link="${name}_link_4"/>
+      <child link="${name}_link_5"/>
+      <origin xyz="0 0 0.1845" rpy="0 0 0"/>
+      <axis xyz="0 0 1"/>
+      <limit lower="${-170 * PI / 180}" upper="${170 * PI / 180}"
+             effort="306" velocity="${velocity_scale_factor * 110 * PI / 180}" />
+      <!-- <safety_controller soft_lower_limit="${-118 * PI / 180}"
+           soft_upper_limit="${118 * PI / 180}"
+           k_position="${safety_controller_k_pos}"
+           k_velocity="${safety_controller_k_vel}"/> -->
+      <dynamics damping="${joint_damping}"/>
+    </joint>
+    <link name="${name}_link_5">
+      <inertial>
+        <origin xyz="0 -0.02 0.104" rpy="0 0 0"/>
+        <mass value="2"/>
+        <inertia ixx="1.84"  ixy="0"  ixz="0" iyy="1.84" iyz="0" izz="0.01" />
+      </inertial>
+      <visual>
+        <origin xyz="0 0 0" rpy="0 0 0"/>
+        <geometry>
+          <mesh filename="package://lbr_iiwa_description/meshes/link_5.stl"/>
+        </geometry>
+        <material name="Orange"/>
+      </visual>
+      <collision>
+        <origin xyz="0 0 0" rpy="0 0 0"/>
+        <geometry>
+          <mesh filename="package://lbr_iiwa_description/meshes/link_5.stl"/>
+        </geometry>
+        <material name="Orange"/>
+      </collision>
+    </link>
+ <!-- joint between link_5 and link_6 -->
+    <joint name="${name}_joint_6" type="revolute">
+      <parent link="${name}_link_5"/>
+      <child link="${name}_link_6"/>
+      <origin xyz="0 -0.0607 0.2155" rpy="0 0 0"/>
+      <axis xyz="0 1 0"/>
+      <limit lower="${-120 * PI / 180}" upper="${120 * PI / 180}"
+             effort="306" velocity="${velocity_scale_factor * 110 * PI / 180}" />
+      <!-- <safety_controller soft_lower_limit="${-118 * PI / 180}"
+           soft_upper_limit="${118 * PI / 180}"
+           k_position="${safety_controller_k_pos}"
+           k_velocity="${safety_controller_k_vel}"/> -->
+      <dynamics damping="${joint_damping}"/>
+    </joint>
+    <link name="${name}_link_6">
+      <inertial>
+        <origin xyz="0 0.06 0" rpy="0 0 0"/>
+        <mass value="2"/>
+        <inertia ixx="0.01"  ixy="0"  ixz="0" iyy="0.01" iyz="0" izz="0.01" />
+      </inertial>
+      <visual>
+        <origin xyz="0 0 0" rpy="0 0 0"/>
+        <geometry>
+          <mesh filename="package://lbr_iiwa_description/meshes/link_6.stl"/>
+        </geometry>
+        <material name="Orange"/>
+      </visual>
+      <collision>
+        <origin xyz="0 0 0" rpy="0 0 0"/>
+        <geometry>
+          <mesh filename="package://lbr_iiwa_description/meshes/link_6.stl"/>
+        </geometry>
+        <material name="Orange"/>
+      </collision>
+    </link>
+ <!-- joint between link_6 and link_7 -->
+    <joint name="${name}_joint_7" type="revolute">
+      <parent link="${name}_link_6"/>
+      <child link="${name}_link_7"/>
+      <origin xyz="0 0.0607 0.0809" rpy="0 0 0"/>
+      <axis xyz="0 0 1"/>
+      <limit lower="${-175 * PI / 180}" upper="${175 * PI / 180}"
+             effort="306" velocity="${velocity_scale_factor * 110 * PI / 180}" />
+      <!-- <safety_controller soft_lower_limit="${-118 * PI / 180}"
+           soft_upper_limit="${118 * PI / 180}"
+           k_position="${safety_controller_k_pos}"
+           k_velocity="${safety_controller_k_vel}"/> -->
+      <dynamics damping="${joint_damping}"/>
+    </joint>
+    <link name="${name}_link_7">
+      <inertial>
+        <origin xyz="0 0 0.02" rpy="0 0 0"/>
+        <mass value="0.5"/>
+        <inertia ixx="0.01"  ixy="0"  ixz="0" iyy="0.01" iyz="0" izz="0.01" />
+      </inertial>
+      <visual>
+        <origin xyz="0 0 0" rpy="0 0 0"/>
+        <geometry>
+          <mesh filename="package://lbr_iiwa_description/meshes/link_7.stl"/>
+        </geometry>
+        <material name="Orange"/>
+      </visual>
+      <collision>
+        <origin xyz="0 0 0" rpy="0 0 0"/>
+        <geometry>
+          <mesh filename="package://lbr_iiwa_description/meshes/link_7.stl"/>
+        </geometry>
+        <material name="Orange"/>
+      </collision>
+    </link>
     <!--Extensions -->
     <xacro:lbr_iiwa_gazebo name="${name}" />

Commit message: works also in rviz now ...

File: lbr_iiwa_description/urdf/lbr_iiwa.xacro (robot description, xacro)
@@ -276,5 +276,5 @@
           <mesh filename="package://lbr_iiwa_description/meshes/link_7.stl"/>
         </geometry>
-        <material name="Orange"/>
+        <material name="Grey"/>
       </visual>
       <collision>
@@ -283,5 +283,5 @@
           <mesh filename="package://lbr_iiwa_description/meshes/link_7.stl"/>
         </geometry>
-        <material name="Orange"/>
+        <material name="Grey"/>
       </collision>
     </link>

Commit message: lbr_iiwa_control: tuned gazebo position controllers

File: lbr_iiwa_description/urdf/lbr_iiwa.xacro (robot description, xacro)
@@ -12,6 +12,7 @@
  <!-- <xacro:property name="safety_controller_k_pos" value="100" />
   <xacro:property name="safety_controller_k_vel" value="2" /> -->
-  <xacro:property name="joint_damping" value="0.1" />
-  <xacro:property name="velocity_scale_factor" value="1"/>
+  <xacro:property name="joint_damping" value="0.5" />
+  <xacro:property name="max_effort" value="300"/>
+  <xacro:property name="max_velocity" value="10"/>
   <!-- right is either 1 (for right arm) or -1 (for left arm) -->
   <xacro:macro name="lbr_iiwa" params="parent name right *origin">
@@ -50,5 +51,5 @@
       <axis xyz="0 0 1"/>
       <limit lower="${-170 * PI / 180}" upper="${170 * PI / 180}"
-             effort="204" velocity="${velocity_scale_factor * 110 * PI / 180}" />
+             effort="${max_effort}" velocity="${max_velocity}" />
       <!--   <safety_controller soft_lower_limit="${-168 * M_PI / 180}"
            soft_upper_limit="${168 * M_PI / 180}"
@@ -85,5 +86,5 @@
       <axis xyz="0 1 0"/>
       <limit lower="${-120 * PI / 180}" upper="${120 * PI / 180}"
-             effort="306" velocity="${velocity_scale_factor * 110 * PI / 180}" />
+             effort="${max_effort}" velocity="${max_velocity}" />
       <!-- <safety_controller soft_lower_limit="${-118 * PI / 180}"
            soft_upper_limit="${118 * PI / 180}"
@@ -120,5 +121,5 @@
       <axis xyz="0 0 1"/>
       <limit lower="${-170 * PI / 180}" upper="${170 * PI / 180}"
-             effort="306" velocity="${velocity_scale_factor * 110 * PI / 180}" />
+             effort="${max_effort}" velocity="${max_velocity}" />
       <!-- <safety_controller soft_lower_limit="${-118 * PI / 180}"
            soft_upper_limit="${118 * PI / 180}"
@@ -155,5 +156,5 @@
       <axis xyz="0 1 0"/>
       <limit lower="${-120 * PI / 180}" upper="${120 * PI / 180}"
-             effort="306" velocity="${velocity_scale_factor * 110 * PI / 180}" />
+             effort="${max_effort}" velocity="${max_velocity}" />
       <!-- <safety_controller soft_lower_limit="${-118 * PI / 180}"
            soft_upper_limit="${118 * PI / 180}"
@@ -190,5 +191,5 @@
       <axis xyz="0 0 1"/>
       <limit lower="${-170 * PI / 180}" upper="${170 * PI / 180}"
-             effort="306" velocity="${velocity_scale_factor * 110 * PI / 180}" />
+             effort="${max_effort}" velocity="${max_velocity}" />
       <!-- <safety_controller soft_lower_limit="${-118 * PI / 180}"
            soft_upper_limit="${118 * PI / 180}"
@@ -201,5 +202,5 @@
         <origin xyz="0 -0.02 0.104" rpy="0 0 0"/>
         <mass value="2"/>
-        <inertia ixx="1.84"  ixy="0"  ixz="0" iyy="1.84" iyz="0" izz="0.01" />
+        <inertia ixx="0.01"  ixy="0"  ixz="0" iyy="0.01" iyz="0" izz="0.01" />
       </inertial>
       <visual>
@@ -225,5 +226,5 @@
       <axis xyz="0 1 0"/>
       <limit lower="${-120 * PI / 180}" upper="${120 * PI / 180}"
-             effort="306" velocity="${velocity_scale_factor * 110 * PI / 180}" />
+             effort="${max_effort}" velocity="${max_velocity}" />
       <!-- <safety_controller soft_lower_limit="${-118 * PI / 180}"
            soft_upper_limit="${118 * PI / 180}"
@@ -260,5 +261,5 @@
       <axis xyz="0 0 1"/>
       <limit lower="${-175 * PI / 180}" upper="${175 * PI / 180}"
-             effort="306" velocity="${velocity_scale_factor * 110 * PI / 180}" />
+             effort="${max_effort}" velocity="${max_velocity}" />
       <!-- <safety_controller soft_lower_limit="${-118 * PI / 180}"
            soft_upper_limit="${118 * PI / 180}"

Commit message: fixed a mesh and tweaked controllers

File: lbr_iiwa_description/urdf/lbr_iiwa.xacro (robot description, xacro)
@@ -200,7 +200,7 @@
     <link name="${name}_link_5">
       <inertial>
-        <origin xyz="0 -0.02 0.104" rpy="0 0 0"/>
-        <mass value="2"/>
-        <inertia ixx="0.01"  ixy="0"  ixz="0" iyy="0.01" iyz="0" izz="0.01" />
+        <origin xyz="0 -0.02 0.08" rpy="0 0 0"/>
+        <mass value="1.7"/>
+        <inertia ixx="0.02"  ixy="0"  ixz="0" iyy="0.02" iyz="0" izz="0.01" />
       </inertial>
       <visual>
@@ -236,6 +236,6 @@
       <inertial>
         <origin xyz="0 0.06 0" rpy="0 0 0"/>
-        <mass value="2"/>
-        <inertia ixx="0.01"  ixy="0"  ixz="0" iyy="0.01" iyz="0" izz="0.01" />
+        <mass value="1.8"/>
+        <inertia ixx="0.01"  ixy="0"  ixz="0" iyy="0.001" iyz="0" izz="0.01" />
       </inertial>
       <visual>
@@ -271,6 +271,6 @@
       <inertial>
         <origin xyz="0 0 0.02" rpy="0 0 0"/>
-        <mass value="0.5"/>
-        <inertia ixx="0.01"  ixy="0"  ixz="0" iyy="0.01" iyz="0" izz="0.01" />
+        <mass value="0.3"/>
+        <inertia ixx="0.001"  ixy="0"  ixz="0" iyy="0.001" iyz="0" izz="0.001" />
       </inertial>
       <visual>

Commit message: lbr_iiwa_description: added finer meshes

File: lbr_iiwa_description/urdf/lbr_iiwa.xacro (robot description, xacro)
@@ -38,5 +38,5 @@
         <origin xyz="0 0 0" rpy="0 0 0"/>
         <geometry>
-          <mesh filename="package://lbr_iiwa_description/meshes/link_0.stl"/>
+          <mesh filename="package://lbr_iiwa_description/meshes/coarse/link_0.stl"/>
         </geometry>
         <material name="Grey"/>
@@ -73,5 +73,5 @@
         <origin xyz="0 0 0" rpy="0 0 0"/>
         <geometry>
-          <mesh filename="package://lbr_iiwa_description/meshes/link_1.stl"/>
+          <mesh filename="package://lbr_iiwa_description/meshes/coarse/link_1.stl"/>
         </geometry>
         <material name="Orange"/>
@@ -108,5 +108,5 @@
         <origin xyz="0 0 0" rpy="0 0 0"/>
         <geometry>
-          <mesh filename="package://lbr_iiwa_description/meshes/link_2.stl"/>
+          <mesh filename="package://lbr_iiwa_description/meshes/coarse/link_2.stl"/>
         </geometry>
         <material name="Orange"/>
@@ -143,5 +143,5 @@
         <origin xyz="0 0 0" rpy="0 0 0"/>
         <geometry>
-          <mesh filename="package://lbr_iiwa_description/meshes/link_3.stl"/>
+          <mesh filename="package://lbr_iiwa_description/meshes/coarse/link_3.stl"/>
         </geometry>
         <material name="Orange"/>
@@ -178,5 +178,5 @@
         <origin xyz="0 0 0" rpy="0 0 0"/>
         <geometry>
-          <mesh filename="package://lbr_iiwa_description/meshes/link_4.stl"/>
+          <mesh filename="package://lbr_iiwa_description/meshes/coarse/link_4.stl"/>
         </geometry>
         <material name="Orange"/>
@@ -213,5 +213,5 @@
         <origin xyz="0 0 0" rpy="0 0 0"/>
         <geometry>
-          <mesh filename="package://lbr_iiwa_description/meshes/link_5.stl"/>
+          <mesh filename="package://lbr_iiwa_description/meshes/coarse/link_5.stl"/>
         </geometry>
         <material name="Orange"/>
@@ -248,5 +248,5 @@
         <origin xyz="0 0 0" rpy="0 0 0"/>
         <geometry>
-          <mesh filename="package://lbr_iiwa_description/meshes/link_6.stl"/>
+          <mesh filename="package://lbr_iiwa_description/meshes/coarse/link_6.stl"/>
         </geometry>
         <material name="Orange"/>
@@ -283,5 +283,5 @@
         <origin xyz="0 0 0" rpy="0 0 0"/>
         <geometry>
-          <mesh filename="package://lbr_iiwa_description/meshes/link_7.stl"/>
+          <mesh filename="package://lbr_iiwa_description/meshes/coarse/link_7.stl"/>
         </geometry>
         <material name="Grey"/>

Commit message: lbr_iiwa_escription: added exemplary self collision tag in the xacro

File: lbr_iiwa_description/urdf/lbr_iiwa.xacro (robot description, xacro)
@@ -40,4 +40,10 @@
         <material name="Grey"/>
       </collision>
+      <self_collision_checking>
+        <origin xyz="0 0 0" rpy="0 0 0"/>
+        <geometry>
+          <capsule radius="0.15" length="0.25"/>
+        </geometry>
+      </self_collision_checking>
     </link>
     <!-- joint between link_0 and link_1 -->

Commit message: lbr_iiwa_description: urdf uses DH - convention now

File: lbr_iiwa_description/urdf/lbr_iiwa.xacro (robot description, xacro)
@@ -86,6 +86,6 @@
       <parent link="${name}_link_1"/>
       <child link="${name}_link_2"/>
-      <origin xyz="0 0 0.2025" rpy="0 0 0"/>
-      <axis xyz="0 1 0"/>
+      <origin xyz="0 0 0.2025" rpy="${PI / 2}   0 ${PI}"/>
+      <axis xyz="0 0 1"/>
       <limit lower="${-120 * PI / 180}" upper="${120 * PI / 180}"
              effort="${max_effort}" velocity="${max_velocity}" />
@@ -98,7 +98,7 @@
     <link name="${name}_link_2">
       <inertial>
-        <origin xyz="0 0.04 0.06" rpy="0 0 0"/>
+        <origin xyz="0.0003 0.059 0.042" rpy="0 0 0"/>
         <mass value="4"/>
-        <inertia ixx="0.05"  ixy="0"  ixz="0" iyy="0.04" iyz="0" izz="0.02" />
+        <inertia ixx="0.05"  ixy="0"  ixz="0" iyy="0.018" iyz="0" izz="0.044" />
       </inertial>
       <visual>
@@ -121,5 +121,5 @@
       <parent link="${name}_link_2"/>
       <child link="${name}_link_3"/>
-      <origin xyz="0 0 0.2045" rpy="0 0 0"/>
+      <origin xyz="0 0.2045 0" rpy="${PI / 2} 0 ${PI}"/>
       <axis xyz="0 0 1"/>
       <limit lower="${-170 * PI / 180}" upper="${170 * PI / 180}"
@@ -135,5 +135,5 @@
         <origin xyz="0 0.03 0.13" rpy="0 0 0"/>
         <mass value="3"/>
-        <inertia ixx="0.08"  ixy="0"  ixz="0" iyy="0.07" iyz="0" izz="0.01" />
+        <inertia ixx="0.08"  ixy="0"  ixz="0" iyy="0.075" iyz="0" izz="0.01" />
       </inertial>
       <visual>
@@ -156,6 +156,6 @@
       <parent link="${name}_link_3"/>
       <child link="${name}_link_4"/>
-      <origin xyz="0 0 0.2155" rpy="0 0 0"/>
-      <axis xyz="0 1 0"/>
+      <origin xyz="0 0 0.2155" rpy="${PI / 2} 0 0"/>
+      <axis xyz="0 0 1"/>
       <limit lower="${-120 * PI / 180}" upper="${120 * PI / 180}"
              effort="${max_effort}" velocity="${max_velocity}" />
@@ -168,7 +168,7 @@
     <link name="${name}_link_4">
       <inertial>
-        <origin xyz="0 -0.03 0.07" rpy="0 0 0"/>
-        <mass value="2.5"/>
-        <inertia ixx="0.03"  ixy="0"  ixz="0" iyy="0.03" iyz="0" izz="0.01" />
+        <origin xyz="0 0.067 0.034" rpy="0 0 0"/>
+        <mass value="2.7"/>
+        <inertia ixx="0.03"  ixy="0"  ixz="0" iyy="0.01" iyz="0" izz="0.029" />
       </inertial>
       <visual>
@@ -191,5 +191,5 @@
       <parent link="${name}_link_4"/>
       <child link="${name}_link_5"/>
-      <origin xyz="0 0 0.1845" rpy="0 0 0"/>
+      <origin xyz="0 0.1845 0" rpy="${-PI / 2} 0 0"/>
       <axis xyz="0 0 1"/>
       <limit lower="${-170 * PI / 180}" upper="${170 * PI / 180}"
@@ -203,7 +203,7 @@
     <link name="${name}_link_5">
       <inertial>
-        <origin xyz="0 -0.02 0.08" rpy="0 0 0"/>
+        <origin xyz="0.0001 0.021 0.076" rpy="0 0 0"/>
         <mass value="1.7"/>
-        <inertia ixx="0.02"  ixy="0"  ixz="0" iyy="0.02" iyz="0" izz="0.01" />
+        <inertia ixx="0.02"  ixy="0"  ixz="0" iyy="0.018" iyz="0" izz="0.005" />
       </inertial>
       <visual>
@@ -226,6 +226,6 @@
       <parent link="${name}_link_5"/>
       <child link="${name}_link_6"/>
-      <origin xyz="0 -0.0607 0.2155" rpy="0 0 0"/>
-      <axis xyz="0 1 0"/>
+      <origin xyz="0 0 0.2155" rpy="${PI / 2} 0 0"/>
+      <axis xyz="0 0 1"/>
       <limit lower="${-120 * PI / 180}" upper="${120 * PI / 180}"
              effort="${max_effort}" velocity="${max_velocity}" />
@@ -238,7 +238,7 @@
     <link name="${name}_link_6">
       <inertial>
-        <origin xyz="0 0.06 0" rpy="0 0 0"/>
+        <origin xyz="0 0.0006 0.0004" rpy="0 0 0"/>
         <mass value="1.8"/>
-        <inertia ixx="0.01"  ixy="0"  ixz="0" iyy="0.001" iyz="0" izz="0.01" />
+        <inertia ixx="0.005"  ixy="0"  ixz="0" iyy="0.0036" iyz="0" izz="0.0047" />
       </inertial>
       <visual>
@@ -261,5 +261,5 @@
       <parent link="${name}_link_6"/>
       <child link="${name}_link_7"/>
-      <origin xyz="0 0.0607 0.0809" rpy="0 0 0"/>
+      <origin xyz="0 0.081 0" rpy="${- PI / 2} ${PI} 0"/>
       <axis xyz="0 0 1"/>
       <limit lower="${-175 * PI / 180}" upper="${175 * PI / 180}"

Commit message: lbr_iiwa_description: fixed bug in urdf

File: lbr_iiwa_description/urdf/lbr_iiwa.xacro (robot description, xacro)
@@ -191,5 +191,5 @@
       <parent link="${name}_link_4"/>
       <child link="${name}_link_5"/>
-      <origin xyz="0 0.1845 0" rpy="${-PI / 2} 0 0"/>
+      <origin xyz="0 0.1845 0" rpy="${-PI / 2} ${PI} 0"/>
       <axis xyz="0 0 1"/>
       <limit lower="${-170 * PI / 180}" upper="${170 * PI / 180}"
