Commit message: GAZEBO : working with new urdf and lauch files
Former-commit-id: fd91439ac2396c52c2a3a95be121427cacf608d0

File: iiwa_description/urdf/iiwa.gazebo.xacro (robot description, xacro)
@@ -1,5 +1,11 @@
 <?xml version="1.0"?>
-<robot name="iiwa" xmlns:xacro="http://www.ros.org/wiki/xacro">
-  <xacro:macro name="iiwa_gazebo" params="name">
+<robot xmlns:xacro="http://www.ros.org/wiki/xacro">
+  <xacro:macro name="iiwa_gazebo" params="name robot_name">
+    <!-- Load Gazebo lib and set the robot namespace -->
+    <gazebo>
+      <plugin name="gazebo_ros_controller" filename="libgazebo_ros_control.so">
+	<robotNamespace>/${robot_name}</robotNamespace>
+      </plugin>
+    </gazebo>
     <!-- Link0 -->
     <gazebo reference="${name}_link_0">

File: iiwa_description/urdf/iiwa.transmission.xacro (robot description, xacro)
@@ -1,4 +1,4 @@
 <?xml version="1.0"?>
-<robot name="iiwa" xmlns:xacro="http://www.ros.org/wiki/xacro">
+<robot xmlns:xacro="http://www.ros.org/wiki/xacro">
   <xacro:macro name="iiwa_transmission" params="name hardware_interface">
     <transmission name="${name}_tran_1">

File: iiwa_description/urdf/utilities.xacro (robot description, xacro)
@@ -1,4 +1,4 @@
 <?xml version="1.0"?>
-<robot name="iiwa" xmlns:xacro="http://www.ros.org/wiki/xacro">
+<robot xmlns:xacro="http://www.ros.org/wiki/xacro">
   <xacro:property name="PI" value="3.1415926535897931"/>
 <!-- The following macros are adapted from the LWR 4 definitions of the RCPRG - https://github.com/RCPRG-ros-pkg/lwr_robot -->

Commit message: Everything seems working with Gazebo!
Former-commit-id: ed6bfbfb836695a862b60eff02582342a05e9c07

File: iiwa_description/urdf/iiwa.gazebo.xacro (robot description, xacro)
@@ -9,5 +9,5 @@
     </gazebo>
     <!-- Link0 -->
-    <gazebo reference="${name}_link_0">
+    <gazebo reference="iiwa_link_0">
       <material>Gazebo/Grey</material>
       <mu1>0.2</mu1>
@@ -15,5 +15,5 @@
     </gazebo>
     <!-- Link1 -->
-    <gazebo reference="${name}_link_1">
+    <gazebo reference="iiwa_link_1">
       <material>Gazebo/Orange</material>
       <mu1>0.2</mu1>
@@ -21,5 +21,5 @@
     </gazebo>
     <!-- Link2 -->
-    <gazebo reference="${name}_link_2">
+    <gazebo reference="iiwa_link_2">
       <material>Gazebo/Orange</material>
       <mu1>0.2</mu1>
@@ -27,5 +27,5 @@
     </gazebo>
     <!-- Link3 -->
-    <gazebo reference="${name}_link_3">
+    <gazebo reference="iiwa_link_3">
       <material>Gazebo/Orange</material>
       <mu1>0.2</mu1>
@@ -33,5 +33,5 @@
     </gazebo>
     <!-- Link4 -->
-    <gazebo reference="${name}_link_4">
+    <gazebo reference="iiwa_link_4">
       <material>Gazebo/Orange</material>
       <mu1>0.2</mu1>
@@ -39,5 +39,5 @@
     </gazebo>
     <!-- Link5 -->
-    <gazebo reference="${name}_link_5">
+    <gazebo reference="iiwa_link_5">
       <material>Gazebo/Orange</material>
       <mu1>0.2</mu1>
@@ -45,5 +45,5 @@
     </gazebo>
     <!-- Link6 -->
-    <gazebo reference="${name}_link_6">
+    <gazebo reference="iiwa_link_6">
       <material>Gazebo/Orange</material>
       <mu1>0.2</mu1>
@@ -51,5 +51,5 @@
     </gazebo>
     <!-- Link7 -->
-    <gazebo reference="${name}_link_7">
+    <gazebo reference="iiwa_link_7">
       <material>Gazebo/Grey</material>
       <mu1>0.2</mu1>

File: iiwa_description/urdf/iiwa.transmission.xacro (robot description, xacro)
@@ -2,70 +2,70 @@
 <robot xmlns:xacro="http://www.ros.org/wiki/xacro">
   <xacro:macro name="iiwa_transmission" params="name hardware_interface">
-    <transmission name="${name}_tran_1">
+    <transmission name="iiwa_tran_1">
       <type>transmission_interface/SimpleTransmission</type>
-      <joint name="${name}_joint_1">
+      <joint name="iiwa_joint_1">
 	<hardwareInterface>${hardware_interface}</hardwareInterface>
       </joint>
-      <actuator name="${name}_motor_1">
+      <actuator name="iiwa_motor_1">
 	<hardwareInterface>${hardware_interface}</hardwareInterface>
 	<mechanicalReduction>1</mechanicalReduction>
       </actuator>
     </transmission>
-    <transmission name="${name}_tran_2">
+    <transmission name="iiwa_tran_2">
       <type>transmission_interface/SimpleTransmission</type>
-      <joint name="${name}_joint_2">
+      <joint name="iiwa_joint_2">
 	<hardwareInterface>${hardware_interface}</hardwareInterface>
       </joint>
-      <actuator name="${name}_motor_2">
+      <actuator name="iiwa_motor_2">
 	<hardwareInterface>${hardware_interface}</hardwareInterface>
 	<mechanicalReduction>1</mechanicalReduction>
       </actuator>
     </transmission>
-    <transmission name="${name}_tran_3">
+    <transmission name="iiwa_tran_3">
       <type>transmission_interface/SimpleTransmission</type>
-      <joint name="${name}_joint_3">
+      <joint name="iiwa_joint_3">
 	<hardwareInterface>${hardware_interface}</hardwareInterface>
       </joint>
-      <actuator name="${name}_motor_3">
+      <actuator name="iiwa_motor_3">
 	<hardwareInterface>${hardware_interface}</hardwareInterface>
 	<mechanicalReduction>1</mechanicalReduction>
       </actuator>
     </transmission>
-    <transmission name="${name}_tran_4">
+    <transmission name="iiwa_tran_4">
       <type>transmission_interface/SimpleTransmission</type>
-      <joint name="${name}_joint_4">
+      <joint name="iiwa_joint_4">
 	<hardwareInterface>${hardware_interface}</hardwareInterface>
       </joint>
-      <actuator name="${name}_motor_4">
+      <actuator name="iiwa_motor_4">
 	<hardwareInterface>${hardware_interface}</hardwareInterface>
 	<mechanicalReduction>1</mechanicalReduction>
       </actuator>
     </transmission>
-    <transmission name="${name}_tran_5">
+    <transmission name="iiwa_tran_5">
       <type>transmission_interface/SimpleTransmission</type>
-      <joint name="${name}_joint_5">
+      <joint name="iiwa_joint_5">
 	<hardwareInterface>${hardware_interface}</hardwareInterface>
       </joint>
-      <actuator name="${name}_motor_5">
+      <actuator name="iiwa_motor_5">
 	<hardwareInterface>${hardware_interface}</hardwareInterface>
 	<mechanicalReduction>1</mechanicalReduction>
       </actuator>
     </transmission>
-    <transmission name="${name}_tran_6">
+    <transmission name="iiwa_tran_6">
       <type>transmission_interface/SimpleTransmission</type>
-      <joint name="${name}_joint_6">
+      <joint name="iiwa_joint_6">
 	<hardwareInterface>${hardware_interface}</hardwareInterface>
       </joint>
-      <actuator name="${name}_motor_6">
+      <actuator name="iiwa_motor_6">
 	<hardwareInterface>${hardware_interface}</hardwareInterface>
 	<mechanicalReduction>1</mechanicalReduction>
       </actuator>
     </transmission>
-    <transmission name="${name}_tran_7">
+    <transmission name="iiwa_tran_7">
       <type>transmission_interface/SimpleTransmission</type>
-      <joint name="${name}_joint_7">
+      <joint name="iiwa_joint_7">
 	<hardwareInterface>${hardware_interface}</hardwareInterface>
       </joint>
-      <actuator name="${name}_motor_7">
+      <actuator name="iiwa_motor_7">
 	<hardwareInterface>${hardware_interface}</hardwareInterface>
 	<mechanicalReduction>1</mechanicalReduction>

Commit message: iiwa7 urdf complete
Former-commit-id: 575317ccd1babd11a53218c1d24bc93490a0ce92

File: iiwa_description/urdf/iiwa.gazebo.xacro (robot description, xacro)
@@ -1,5 +1,5 @@
 <?xml version="1.0"?>
 <robot xmlns:xacro="http://www.ros.org/wiki/xacro">
-  <xacro:macro name="iiwa_gazebo" params="name robot_name">
+  <xacro:macro name="iiwa_gazebo" params="robot_name">
     <!-- Load Gazebo lib and set the robot namespace -->
     <gazebo>

File: iiwa_description/urdf/iiwa.transmission.xacro (robot description, xacro)
@@ -1,5 +1,5 @@
 <?xml version="1.0"?>
 <robot xmlns:xacro="http://www.ros.org/wiki/xacro">
-  <xacro:macro name="iiwa_transmission" params="name hardware_interface">
+  <xacro:macro name="iiwa_transmission" params="hardware_interface">
     <transmission name="iiwa_tran_1">
       <type>transmission_interface/SimpleTransmission</type>

File: iiwa_description/urdf/iiwa14.urdf.xacro (robot description, xacro)
@@ -8,5 +8,5 @@
   <link name="world"/>
   <!--iiwa-->
-  <xacro:iiwa14 name="iiwa14" hardware_interface="$(arg hardware_interface)" robot_name="$(arg robot_name)" parent="world">
+  <xacro:iiwa14 hardware_interface="$(arg hardware_interface)" robot_name="$(arg robot_name)" parent="world">
     <origin xyz="0 0 0.0" rpy="0 0 0" />
   </xacro:iiwa14>

File: iiwa_description/urdf/iiwa14.xacro (robot description, xacro)
@@ -13,5 +13,5 @@
   <xacro:property name="max_effort" value="300"/>
   <xacro:property name="max_velocity" value="10"/>
-  <xacro:macro name="iiwa14" params="parent name hardware_interface robot_name *origin">
+  <xacro:macro name="iiwa14" params="parent hardware_interface robot_name *origin">
     <!--joint between {parent} and link_0-->
     <joint name="${parent}_joint" type="fixed">
@@ -302,6 +302,6 @@
     </link>
     <!--Extensions -->
-    <xacro:iiwa_gazebo name="${name}" robot_name="${robot_name}" />
-    <xacro:iiwa_transmission name="${name}" hardware_interface="${hardware_interface}"/>
+    <xacro:iiwa_gazebo robot_name="${robot_name}" />
+    <xacro:iiwa_transmission hardware_interface="${hardware_interface}"/>
   </xacro:macro>
 </robot>
