Commit message: Final URDF, IIWA7 one is really nice
Former-commit-id: 6bf9ce749043b7c3453f95fb9e26c4417b110402

File: iiwa_description/urdf/iiwa14.urdf.xacro (robot description, xacro)
@@ -8,5 +8,5 @@
   <link name="world"/>
   <!--iiwa-->
-  <xacro:iiwa14 hardware_interface="$(arg hardware_interface)" robot_name="$(arg robot_name)" parent="world">
+  <xacro:iiwa14 hardware_interface="$(arg hardware_interface)" robot_name="$(arg robot_name)" pneumatic="$(arg pneumatic)" parent="world">
     <origin xyz="0 0 0.0" rpy="0 0 0" />
   </xacro:iiwa14>

File: iiwa_description/urdf/iiwa14.xacro (robot description, xacro)
@@ -13,5 +13,8 @@
   <xacro:property name="max_effort" value="300"/>
   <xacro:property name="max_velocity" value="10"/>
-  <xacro:macro name="iiwa14" params="parent hardware_interface robot_name *origin">
+    <!-- Flange lenghts    -->
+  <xacro:property name="basic_flange" value="0.045"/>
+  <xacro:property name="pneumatic_flange" value="0.075"/>
+  <xacro:macro name="iiwa14" params="parent hardware_interface robot_name pneumatic *origin">
     <!--joint between {parent} and link_0-->
     <joint name="${parent}_joint" type="fixed">
@@ -292,9 +295,13 @@
       </collision>
     </link>
-    <!-- joint between link_7 and end effector -->
     <joint name="iiwa_joint_ee" type="fixed">
       <parent link="iiwa_link_7"/>
       <child link="iiwa_link_ee"/>
-      <origin xyz="0 0 0.045" rpy="${PI} ${PI} ${PI}"/>
+      <xacro:if value="${pneumatic}">
+	        <origin xyz="0 0 ${pneumatic_flange}" rpy="${PI} ${PI} ${PI}"/>
+      </xacro:if>
+      <xacro:unless value="${pneumatic}">
+	        <origin xyz="0 0 ${basic_flange}" rpy="${PI} ${PI} ${PI}"/>
+      </xacro:unless>
       <axis xyz="0 0 1"/>
     </joint>

File: iiwa_description/urdf/iiwa7.urdf (robot description, URDF)
Before this commit: robot iiwa7, 10 links, 9 joints
Joints:
- joint iiwa_joint_1: origin xyz=0 0 0.15 rpy=0 0 0 -> xyz=0 0 0.1575 rpy=0 0 0
- joint iiwa_joint_2: origin xyz=0 0 0.19 rpy=1.57079632679   0 3.14159265359 -> xyz=0 -0.0005 0.1840 rpy=1.57079632679   0 3.14159265359
- joint iiwa_joint_3: origin xyz=0 0.20 0 rpy=1.57079632679 0 3.14159265359 -> xyz=0 0.184 0 rpy=1.57079632679 0 3.14159265359
- joint iiwa_joint_4: origin xyz=0 0 0.2 rpy=1.57079632679 0 0 -> xyz=0 0 0.21550 rpy=1.57079632679 0 0
- joint iiwa_joint_5: origin xyz=0 0.20 0 rpy=-1.57079632679 3.14159265359 0 -> xyz=0 0.1840 0 rpy=-1.57079632679 3.14159265359 0
- joint iiwa_joint_6: origin xyz=0 0 0.20 rpy=1.57079632679 0 0 -> xyz=0 0.06070 0.21550 rpy=1.57079632679 0 0
- joint iiwa_joint_7: origin xyz=0 0.081 0 rpy=-1.57079632679 3.14159265359 0 -> xyz=0 0.0805 0.060 rpy=-1.57079632679 3.14159265359 0

File: iiwa_description/urdf/iiwa7.urdf.xacro (robot description, xacro)
@@ -8,5 +8,5 @@
   <link name="world"/>
   <!--iiwa-->
-  <xacro:iiwa7 hardware_interface="$(arg hardware_interface)" robot_name="$(arg robot_name)" flange="$(arg flange)" parent="world">
+  <xacro:iiwa7 hardware_interface="$(arg hardware_interface)" robot_name="$(arg robot_name)" pneumatic="$(arg pneumatic)" parent="world">
     <origin xyz="0 0 0.0" rpy="0 0 0" />
   </xacro:iiwa7>

File: iiwa_description/urdf/iiwa7.xacro (robot description, xacro)
@@ -13,5 +13,8 @@
   <xacro:property name="max_effort" value="300"/>
   <xacro:property name="max_velocity" value="10"/>
-  <xacro:macro name="iiwa7" params="parent hardware_interface robot_name flange *origin">
+  <!-- Flange lenghts    -->
+  <xacro:property name="basic_flange" value="0.045"/>
+  <xacro:property name="pneumatic_flange" value="0.075"/>
+  <xacro:macro name="iiwa7" params="parent hardware_interface robot_name pneumatic *origin">
     <!--joint between {parent} and link_0-->
     <joint name="${parent}_joint" type="fixed">
@@ -51,5 +54,5 @@
       <parent link="iiwa_link_0"/>
       <child link="iiwa_link_1"/>
-      <origin xyz="0 0 0.15" rpy="0 0 0"/>
+      <origin xyz="0 0 0.1575" rpy="0 0 0"/>
       <axis xyz="0 0 1"/>
       <limit lower="${-170 * PI / 180}" upper="${170 * PI / 180}"
@@ -68,5 +71,5 @@
       </inertial>
       <visual>
-        <origin xyz="0 0 -0.003" rpy="0 0 0"/>
+        <origin xyz="0 0 0" rpy="0 0 0"/>
         <geometry>
           <mesh filename="package://iiwa_description/meshes/iiwa7/visual/link_1.stl"/>
@@ -75,5 +78,5 @@
       </visual>
       <collision>
-        <origin xyz="0 0 -0.003" rpy="0 0 0"/>
+        <origin xyz="0 0 0" rpy="0 0 0"/>
         <geometry>
           <mesh filename="package://iiwa_description/meshes/iiwa7/collision/link_1.stl"/>
@@ -82,9 +85,8 @@
       </collision>
     </link>
-    <!-- joint between link_1 and link_2 -->
     <joint name="iiwa_joint_2" type="revolute">
       <parent link="iiwa_link_1"/>
       <child link="iiwa_link_2"/>
-      <origin xyz="0 0 0.19" rpy="${PI / 2}   0 ${PI}"/>
+      <origin xyz="0 -0.0005 0.1840" rpy="${PI / 2}   0 ${PI}"/>
       <axis xyz="0 0 1"/>
       <limit lower="${-120 * PI / 180}" upper="${120 * PI / 180}"
@@ -117,9 +119,8 @@
       </collision>
     </link>
-    <!-- joint between link_2 and link_3 -->
     <joint name="iiwa_joint_3" type="revolute">
       <parent link="iiwa_link_2"/>
       <child link="iiwa_link_3"/>
-      <origin xyz="0 0.20 0" rpy="${PI / 2} 0 ${PI}"/>
+      <origin xyz="0 0.184 0" rpy="${PI / 2} 0 ${PI}"/>
       <axis xyz="0 0 1"/>
       <limit lower="${-170 * PI / 180}" upper="${170 * PI / 180}"
@@ -138,5 +139,5 @@
       </inertial>
       <visual>
-        <origin xyz="0 0 -0.02" rpy="0 0 0"/>
+        <origin xyz="0 0 0" rpy="0 0 0"/>
         <geometry>
           <mesh filename="package://iiwa_description/meshes/iiwa7/visual/link_3.stl"/>
@@ -145,5 +146,5 @@
       </visual>
       <collision>
-        <origin xyz="0 0 -0.02" rpy="0 0 0"/>
+        <origin xyz="0 0 0" rpy="0 0 0"/>
         <geometry>
           <mesh filename="package://iiwa_description/meshes/iiwa7/collision/link_3.stl"/>
@@ -152,9 +153,8 @@
       </collision>
     </link>
-   <!-- joint between link_3 and link_4 -->
     <joint name="iiwa_joint_4" type="revolute">
       <parent link="iiwa_link_3"/>
       <child link="iiwa_link_4"/>
-      <origin xyz="0 0 0.2" rpy="${PI / 2} 0 0"/>
+      <origin xyz="0 0 0.21550" rpy="${PI / 2} 0 0"/>
       <axis xyz="0 0 1"/>
       <limit lower="${-120 * PI / 180}" upper="${120 * PI / 180}"
@@ -173,5 +173,5 @@
       </inertial>
       <visual>
-        <origin xyz="0 -0.005 0" rpy="0 0 0"/>
+        <origin xyz="0 0 0" rpy="0 0 0"/>
         <geometry>
           <mesh filename="package://iiwa_description/meshes/iiwa7/visual/link_4.stl"/>
@@ -180,5 +180,5 @@
       </visual>
       <collision>
-        <origin xyz="0 -0.005 0" rpy="0 0 0"/>
+        <origin xyz="0 0 0" rpy="0 0 0"/>
         <geometry>
           <mesh filename="package://iiwa_description/meshes/iiwa7/collision/link_4.stl"/>
@@ -187,9 +187,8 @@
       </collision>
     </link>
-    <!-- joint between link_4 and link_5 -->
     <joint name="iiwa_joint_5" type="revolute">
       <parent link="iiwa_link_4"/>
       <child link="iiwa_link_5"/>
-      <origin xyz="0 0.20 0" rpy="${-PI / 2} ${PI} 0"/>
+      <origin xyz="0 0.1840 0" rpy="${-PI / 2} ${PI} 0"/>
       <axis xyz="0 0 1"/>
       <limit lower="${-170 * PI / 180}" upper="${170 * PI / 180}"
@@ -208,5 +207,5 @@
       </inertial>
       <visual>
-        <origin xyz="0 0 -0.022" rpy="0 0 0"/>
+        <origin xyz="0 0 0" rpy="0 0 0"/>
         <geometry>
           <mesh filename="package://iiwa_description/meshes/iiwa7/visual/link_5.stl"/>
@@ -215,5 +214,5 @@
       </visual>
       <collision>
-        <origin xyz="0 0 -0.022" rpy="0 0 0"/>
+        <origin xyz="0 0 0" rpy="0 0 0"/>
         <geometry>
           <mesh filename="package://iiwa_description/meshes/iiwa7/collision/link_5.stl"/>
@@ -222,9 +221,8 @@
       </collision>
     </link>
- <!-- joint between link_5 and link_6 -->
     <joint name="iiwa_joint_6" type="revolute">
       <parent link="iiwa_link_5"/>
       <child link="iiwa_link_6"/>
-      <origin xyz="0 0 0.20" rpy="${PI / 2} 0 0"/>
+      <origin xyz="0 0.06070 0.21550" rpy="${PI / 2} 0 0"/>
       <axis xyz="0 0 1"/>
       <limit lower="${-120 * PI / 180}" upper="${120 * PI / 180}"
@@ -243,5 +241,5 @@
       </inertial>
       <visual>
-        <origin xyz="0 -0.005 0" rpy="0 0 0"/>
+        <origin xyz="0 0 0" rpy="0 0 0"/>
         <geometry>
           <mesh filename="package://iiwa_description/meshes/iiwa7/visual/link_6.stl"/>
@@ -250,5 +248,5 @@
       </visual>
       <collision>
-        <origin xyz="0 -0.005 0" rpy="0 0 0"/>
+        <origin xyz="0 0 0" rpy="0 0 0"/>
         <geometry>
           <mesh filename="package://iiwa_description/meshes/iiwa7/collision/link_6.stl"/>
@@ -257,9 +255,8 @@
       </collision>
     </link>
- <!-- joint between link_6 and link_7 -->
     <joint name="iiwa_joint_7" type="revolute">
       <parent link="iiwa_link_6"/>
       <child link="iiwa_link_7"/>
-      <origin xyz="0 0.081 0" rpy="${- PI / 2} ${PI} 0"/>
+      <origin xyz="0 0.0805 0.060" rpy="${- PI / 2} ${PI} 0"/>
       <axis xyz="0 0 1"/>
       <limit lower="${-175 * PI / 180}" upper="${175 * PI / 180}"
@@ -278,23 +275,27 @@
       </inertial>
       <visual>
-        <origin xyz="-0.053 -0.05 -0.005" rpy="0 0 0"/>
-        <geometry>
-          <mesh filename="package://iiwa_description/meshes/iiwa7/visual/link_7_${flange}.stl"/>
+        <origin xyz="0 0 0" rpy="0 0 0"/>
+        <geometry>
+          <mesh filename="package://iiwa_description/meshes/iiwa7/visual/link_7_basic.stl"/>
         </geometry>
         <material name="Grey"/>
       </visual>
       <collision>
-        <origin xyz="-0.053 -0.05 -0.005" rpy="0 0 0"/>
-        <geometry>
-          <mesh filename="package://iiwa_description/meshes/iiwa7/collision/link_7_${flange}.stl"/>
+        <origin xyz="0 0 0" rpy="0 0 0"/>
+        <geometry>
+          <mesh filename="package://iiwa_description/meshes/iiwa7/collision/link_7_basic.stl"/>
         </geometry>
         <material name="Grey"/>
       </collision>
     </link>
-     <!-- joint between link_7 and end effector -->
     <joint name="iiwa_joint_ee" type="fixed">
       <parent link="iiwa_link_7"/>
       <child link="iiwa_link_ee"/>
-      <origin xyz="0 0 0.045" rpy="${PI} ${PI} ${PI}"/>
+      <xacro:if value="${pneumatic}">
+	        <origin xyz="0 0 ${pneumatic_flange}" rpy="${PI} ${PI} ${PI}"/>
+      </xacro:if>
+      <xacro:unless value="${pneumatic}">
+	        <origin xyz="0 0 ${basic_flange}" rpy="${PI} ${PI} ${PI}"/>
+      </xacro:unless>
       <axis xyz="0 0 1"/>
     </joint>

Commit message: All the flanges have the same length...pneumatic is 0.1mm longer. Removed that option for the moment. iiwa7 is the default for moveit now.
Former-commit-id: 00ed7c7180c669dc2c85d284072782ea07c48583

File: iiwa_description/urdf/iiwa14.urdf.xacro (robot description, xacro)
@@ -8,5 +8,5 @@
   <link name="world"/>
   <!--iiwa-->
-  <xacro:iiwa14 hardware_interface="$(arg hardware_interface)" robot_name="$(arg robot_name)" pneumatic="$(arg pneumatic)" parent="world">
+  <xacro:iiwa14 hardware_interface="$(arg hardware_interface)" robot_name="$(arg robot_name)" parent="world">
     <origin xyz="0 0 0.0" rpy="0 0 0" />
   </xacro:iiwa14>

File: iiwa_description/urdf/iiwa14.xacro (robot description, xacro)
@@ -13,8 +13,5 @@
   <xacro:property name="max_effort" value="300"/>
   <xacro:property name="max_velocity" value="10"/>
-    <!-- Flange lenghts    -->
-  <xacro:property name="basic_flange" value="0.045"/>
-  <xacro:property name="pneumatic_flange" value="0.075"/>
-  <xacro:macro name="iiwa14" params="parent hardware_interface robot_name pneumatic *origin">
+  <xacro:macro name="iiwa14" params="parent hardware_interface robot_name *origin">
     <!--joint between {parent} and link_0-->
     <joint name="${parent}_joint" type="fixed">
@@ -298,10 +295,5 @@
       <parent link="iiwa_link_7"/>
       <child link="iiwa_link_ee"/>
-      <xacro:if value="${pneumatic}">
-	        <origin xyz="0 0 ${pneumatic_flange}" rpy="${PI} ${PI} ${PI}"/>
-      </xacro:if>
-      <xacro:unless value="${pneumatic}">
-	        <origin xyz="0 0 ${basic_flange}" rpy="${PI} ${PI} ${PI}"/>
-      </xacro:unless>
+      <origin xyz="0 0 0.045" rpy="${PI} ${PI} ${PI}"/>
       <axis xyz="0 0 1"/>
     </joint>

File: iiwa_description/urdf/iiwa7.urdf.xacro (robot description, xacro)
@@ -8,5 +8,5 @@
   <link name="world"/>
   <!--iiwa-->
-  <xacro:iiwa7 hardware_interface="$(arg hardware_interface)" robot_name="$(arg robot_name)" pneumatic="$(arg pneumatic)" parent="world">
+  <xacro:iiwa7 hardware_interface="$(arg hardware_interface)" robot_name="$(arg robot_name)" parent="world">
     <origin xyz="0 0 0.0" rpy="0 0 0" />
   </xacro:iiwa7>

File: iiwa_description/urdf/iiwa7.xacro (robot description, xacro)
@@ -13,8 +13,5 @@
   <xacro:property name="max_effort" value="300"/>
   <xacro:property name="max_velocity" value="10"/>
-  <!-- Flange lenghts    -->
-  <xacro:property name="basic_flange" value="0.045"/>
-  <xacro:property name="pneumatic_flange" value="0.075"/>
-  <xacro:macro name="iiwa7" params="parent hardware_interface robot_name pneumatic *origin">
+  <xacro:macro name="iiwa7" params="parent hardware_interface robot_name *origin">
     <!--joint between {parent} and link_0-->
     <joint name="${parent}_joint" type="fixed">
@@ -292,10 +289,5 @@
       <parent link="iiwa_link_7"/>
       <child link="iiwa_link_ee"/>
-      <xacro:if value="${pneumatic}">
-	        <origin xyz="0 0 ${pneumatic_flange}" rpy="${PI} ${PI} ${PI}"/>
-      </xacro:if>
-      <xacro:unless value="${pneumatic}">
-	        <origin xyz="0 0 ${basic_flange}" rpy="${PI} ${PI} ${PI}"/>
-      </xacro:unless>
+      <origin xyz="0 0 0.045" rpy="${PI} ${PI} ${PI}"/>
       <axis xyz="0 0 1"/>
     </joint>
