Commit message: Full parametrized : hardware_interface, robot_name, mode, flange, trajectory controllers.
GAZEBO : IIWA14 is working good, weird behaviour using effort/velocity controllers should be due to the almost random controllers' parameters.
IIWA7 is not working, the model is shaking all the time. Maybe due to the inertia values taken from the IIWA14 URDF?

MOVEIT : everything looks good, to test with the real robot.


Former-commit-id: 9110c65c742500d5323a73a51529b1a9da41ef07

File: iiwa_description/urdf/iiwa14.urdf (robot description, URDF)
Before this commit: robot iiwa14, 10 links, 9 joints
Links:
- removed link iiwa14_link_0
- removed link iiwa14_link_1
- removed link iiwa14_link_2
- removed link iiwa14_link_3
- removed link iiwa14_link_4
- removed link iiwa14_link_5
- removed link iiwa14_link_6
- removed link iiwa14_link_7
- removed link iiwa14_link_ee
- added link iiwa_link_0, mass 5; collision mesh filename=package://iiwa_description/meshes/iiwa14/collision/link_0.s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; visual mesh filename=package://iiwa_description/meshes/iiwa14/visual/link_0.stl
- added link iiwa_link_1, mass 4; collision mesh filename=package://iiwa_description/meshes/iiwa14/collision/link_1.s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; visual mesh filename=package://iiwa_description/meshes/iiwa14/visual/link_1.stl
- added link iiwa_link_2, mass 4; collision mesh filename=package://iiwa_description/meshes/iiwa14/collision/link_2.s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; visual mesh filename=package://iiwa_description/meshes/iiwa14/visual/link_2.stl
- added link iiwa_link_3, mass 3; collision mesh filename=package://iiwa_description/meshes/iiwa14/collision/link_3.s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; visual mesh filename=package://iiwa_description/meshes/iiwa14/visual/link_3.stl
- added link iiwa_link_4, mass 2.7; collision mesh filename=package://iiwa_description/meshes/iiwa14/collision/link_4.s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; visual mesh filename=package://iiwa_description/meshes/iiwa14/visual/link_4.stl
- added link iiwa_link_5, mass 1.7; collision mesh filename=package://iiwa_description/meshes/iiwa14/collision/link_5.s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; visual mesh filename=package://iiwa_description/meshes/iiwa14/visual/link_5.stl
- added link iiwa_link_6, mass 1.8; collision mesh filename=package://iiwa_description/meshes/iiwa14/collision/link_6.s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; visual mesh filename=package://iiwa_description/meshes/iiwa14/visual/link_6.stl
- added link iiwa_link_7, mass 0.3; collision mesh filename=package://iiwa_description/meshes/iiwa14/collision/link_7.s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; visual mesh filename=package://iiwa_description/meshes/iiwa14/visual/link_7.stl
- added link iiwa_link_ee
Joints:
- removed joint iiwa14_joint_1
- removed joint iiwa14_joint_2
- removed joint iiwa14_joint_3
- removed joint iiwa14_joint_4
- removed joint iiwa14_joint_5
- removed joint iiwa14_joint_6
- removed joint iiwa14_joint_7
- removed joint iiwa14_joint_ee
- added joint iiwa_joint_1: type revolute, parent iiwa_link_0, child iiwa_link_1, origin xyz=0 0 0.1575 rpy=0 0 0, axis 0 0 1, limit lower=-2.96705972839 upper=2.96705972839 effort=300 velocity=10
- added joint iiwa_joint_2: type revolute, parent iiwa_link_1, child iiwa_link_2, origin xyz=0 0 0.2025 rpy=1.57079632679   0 3.14159265359, axis 0 0 1, limit lower=-2.09439510239 upper=2.09439510239 effort=300 velocity=10
- added joint iiwa_joint_3: type revolute, parent iiwa_link_2, child iiwa_link_3, origin xyz=0 0.2045 0 rpy=1.57079632679 0 3.14159265359, axis 0 0 1, limit lower=-2.96705972839 upper=2.96705972839 effort=300 velocity=10
- added joint iiwa_joint_4: type revolute, parent iiwa_link_3, child iiwa_link_4, origin xyz=0 0 0.2155 rpy=1.57079632679 0 0, axis 0 0 1, limit lower=-2.09439510239 upper=2.09439510239 effort=300 velocity=10
- added joint iiwa_joint_5: type revolute, parent iiwa_link_4, child iiwa_link_5, origin xyz=0 0.1845 0 rpy=-1.57079632679 3.14159265359 0, axis 0 0 1, limit lower=-2.96705972839 upper=2.96705972839 effort=300 velocity=10
- added joint iiwa_joint_6: type revolute, parent iiwa_link_5, child iiwa_link_6, origin xyz=0 0 0.2155 rpy=1.57079632679 0 0, axis 0 0 1, limit lower=-2.09439510239 upper=2.09439510239 effort=300 velocity=10
- added joint iiwa_joint_7: type revolute, parent iiwa_link_6, child iiwa_link_7, origin xyz=0 0.081 0 rpy=-1.57079632679 3.14159265359 0, axis 0 0 1, limit lower=-3.05432619099 upper=3.05432619099 effort=300 velocity=10
- added joint iiwa_joint_ee: type fixed, parent iiwa_link_7, child iiwa_link_ee, origin xyz=0 0 0.045 rpy=3.14159265359 3.14159265359 3.14159265359, axis 0 0 1
- joint world_joint: child iiwa14_link_0 -> iiwa_link_0

File: iiwa_description/urdf/iiwa7.urdf (robot description, URDF)
Before this commit: robot iiwa7, 10 links, 9 joints
Links:
- link iiwa_link_7: geometry collision mesh filename=package://iiwa_description/meshes/iiwa7/collision/link_7_ba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; visual mesh filename=package://iiwa_description/meshes/iiwa7/visual/link_7_basic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

Commit message: updated URDF. added tool0 frame as endeffector, with X point upwards

File: iiwa_description/urdf/iiwa14.urdf (robot description, URDF)
Before this commit: robot iiwa14, 10 links, 9 joints
Links:
- added link tool0
Joints:
- removed joint world_joint
- added joint tool0_joint: type fixed, parent iiwa_link_ee, child tool0, origin xyz=0 0 0 rpy=0 -1.57079632679 0
- added joint world_iiwa_joint: type fixed, parent world, child iiwa_link_0, origin xyz=0 0 0.0 rpy=0 0 0

File: iiwa_description/urdf/iiwa14.xacro (robot description, xacro)
@@ -300,4 +300,11 @@
     <link name="${robot_name}_link_ee">
     </link>
+    <joint name="tool0_joint" type="fixed">
+      <parent link="${robot_name}_link_ee"/>
+      <child link="tool0"/>
+      <origin xyz="0 0 0" rpy="0 -${PI/2} 0"/>
+    </joint>
+    <link name="tool0">
+    </link>
     <!--Extensions -->
     <xacro:iiwa_gazebo robot_name="${robot_name}" />

File: iiwa_description/urdf/iiwa7.urdf (robot description, URDF)
Before this commit: robot iiwa7, 10 links, 9 joints
Links:
- added link tool0
Joints:
- removed joint world_joint
- added joint tool0_joint: type fixed, parent iiwa_link_ee, child tool0, origin xyz=0 0 0 rpy=0 -1.57079632679 0
- added joint world_iiwa_joint: type fixed, parent world, child iiwa_link_0, origin xyz=0 0 0.0 rpy=0 0 0
- joint iiwa_joint_1: origin xyz=0 0 0.1575 rpy=0 0 0 -> xyz=0 0 0.15 rpy=0 0 0
- joint iiwa_joint_2: origin xyz=0 -0.0005 0.1840 rpy=1.57079632679   0 3.14159265359 -> xyz=0 0 0.19 rpy=1.57079632679   0 3.14159265359
- joint iiwa_joint_3: origin xyz=0 0.184 0 rpy=1.57079632679 0 3.14159265359 -> xyz=0 0.21 0 rpy=1.57079632679 0 3.14159265359
- joint iiwa_joint_4: origin xyz=0 0 0.21550 rpy=1.57079632679 0 0 -> xyz=0 0 0.19 rpy=1.57079632679 0 0
- joint iiwa_joint_5: limit lower=-2.96705972839 upper=2.96705972839 effort=300 velocity=10 -> lower=-3.05432619099 upper=3.05432619099 effort=300 velocity=10; origin xyz=0 0.1840 0 rpy=-1.57079632679 3.14159265359 0 -> xyz=0 0.21 0 rpy=-1.57079632679 3.14159265359 0
- joint iiwa_joint_6: origin xyz=0 0.06070 0.21550 rpy=1.57079632679 0 0 -> xyz=0 0.06070 0.19 rpy=1.57079632679 0 0
- joint iiwa_joint_7: origin xyz=0 0.0805 0.060 rpy=-1.57079632679 3.14159265359 0 -> xyz=0 0.081 0.06070 rpy=-1.57079632679 3.14159265359 0

File: iiwa_description/urdf/iiwa7.xacro (robot description, xacro)
@@ -186,5 +186,5 @@
     <joint name="${robot_name}_joint_5" type="revolute">
       <parent link="${robot_name}_link_4"/>
-      <child link="${robot_name}_link_5"/>-169
+      <child link="${robot_name}_link_5"/>
       <origin xyz="0 0.21 0" rpy="${-PI / 2} ${PI} 0"/>
       <axis xyz="0 0 1"/>
@@ -293,4 +293,11 @@
     </joint>
     <link name="${robot_name}_link_ee">
+    </link>
+    <joint name="tool0_joint" type="fixed">
+      <parent link="${robot_name}_link_ee"/>
+      <child link="tool0"/>
+      <origin xyz="0 0 0" rpy="0 -${PI/2} 0"/>
+    </joint>
+    <link name="tool0">
     </link>
     <!--Extensions -->

Commit message: fixed last fixed joint and last 2 links now there is one endeffector link with a coordinate frame as the one use by kuka (z axis upwards) and one with the convention used by ROS (x axis upwards)

File: iiwa_description/urdf/iiwa14.urdf (robot description, URDF)
Before this commit: robot iiwa14, 11 links, 10 joints
Links:
- removed link tool0
- added link iiwa_link_ee_kuka
Joints:
- joint iiwa_joint_ee: child iiwa_link_ee -> iiwa_link_ee_kuka
- joint tool0_joint: child tool0 -> iiwa_link_ee; origin xyz=0 0 0 rpy=0 -1.57079632679 0 -> xyz=0 0 0.045 rpy=0 -1.57079632679 0; parent iiwa_link_ee -> iiwa_link_7

File: iiwa_description/urdf/iiwa14.xacro (robot description, xacro)
@@ -294,16 +294,16 @@
     <joint name="${robot_name}_joint_ee" type="fixed">
       <parent link="${robot_name}_link_7"/>
+      <child link="${robot_name}_link_ee_kuka"/>
+      <origin xyz="0 0 0.045" rpy="${PI} ${PI} ${PI}"/>
+      <axis xyz="0 0 1"/>
+    </joint>
+    <link name="${robot_name}_link_ee_kuka">
+    </link>
+    <joint name="tool0_joint" type="fixed">
+      <parent link="${robot_name}_link_7"/>
       <child link="${robot_name}_link_ee"/>
-      <origin xyz="0 0 0.045" rpy="${PI} ${PI} ${PI}"/>
-      <axis xyz="0 0 1"/>
+      <origin xyz="0 0 0.045" rpy="0 -${PI/2} 0"/>
     </joint>
     <link name="${robot_name}_link_ee">
-    </link>
-    <joint name="tool0_joint" type="fixed">
-      <parent link="${robot_name}_link_ee"/>
-      <child link="tool0"/>
-      <origin xyz="0 0 0" rpy="0 -${PI/2} 0"/>
-    </joint>
-    <link name="tool0">
     </link>
     <!--Extensions -->

File: iiwa_description/urdf/iiwa7.urdf (robot description, URDF)
Before this commit: robot iiwa7, 11 links, 10 joints
Links:
- removed link tool0
- added link iiwa_link_ee_kuka
Joints:
- joint iiwa_joint_ee: child iiwa_link_ee -> iiwa_link_ee_kuka
- joint tool0_joint: child tool0 -> iiwa_link_ee; origin xyz=0 0 0 rpy=0 -1.57079632679 0 -> xyz=0 0 0.045 rpy=0 -1.57079632679 0; parent iiwa_link_ee -> iiwa_link_7

File: iiwa_description/urdf/iiwa7.xacro (robot description, xacro)
@@ -288,16 +288,16 @@
     <joint name="${robot_name}_joint_ee" type="fixed">
       <parent link="${robot_name}_link_7"/>
+      <child link="${robot_name}_link_ee_kuka"/>
+      <origin xyz="0 0 0.045" rpy="${PI} ${PI} ${PI}"/>
+      <axis xyz="0 0 1"/>
+    </joint>
+    <link name="${robot_name}_link_ee_kuka">
+    </link>
+    <joint name="tool0_joint" type="fixed">
+      <parent link="${robot_name}_link_7"/>
       <child link="${robot_name}_link_ee"/>
-      <origin xyz="0 0 0.045" rpy="${PI} ${PI} ${PI}"/>
-      <axis xyz="0 0 1"/>
+      <origin xyz="0 0 0.045" rpy="0 -${PI/2} 0"/>
     </joint>
     <link name="${robot_name}_link_ee">
-    </link>
-    <joint name="tool0_joint" type="fixed">
-      <parent link="${robot_name}_link_ee"/>
-      <child link="tool0"/>
-      <origin xyz="0 0 0" rpy="0 -${PI/2} 0"/>
-    </joint>
-    <link name="tool0">
     </link>
     <!--Extensions -->
