Commit message: fixed name of last joint

File: iiwa_description/urdf/iiwa14.urdf (robot description, URDF)
Before this commit: robot iiwa14, 11 links, 10 joints
Joints:
- removed joint tool0_joint
- added joint iiwa_joint_ee_kuka: type fixed, parent iiwa_link_7, child iiwa_link_ee_kuka, origin xyz=0 0 0.045 rpy=3.14159265359 3.14159265359 3.14159265359, axis 0 0 1
- joint iiwa_joint_ee: axis 0 0 1 -> (none); child iiwa_link_ee_kuka -> iiwa_link_ee; origin xyz=0 0 0.045 rpy=3.14159265359 3.14159265359 3.14159265359 -> xyz=0 0 0.045 rpy=0 -1.57079632679 0

File: iiwa_description/urdf/iiwa14.xacro (robot description, xacro)
@@ -294,4 +294,11 @@
     <joint name="${robot_name}_joint_ee" type="fixed">
       <parent link="${robot_name}_link_7"/>
+      <child link="${robot_name}_link_ee"/>
+      <origin xyz="0 0 0.045" rpy="0 -${PI/2} 0"/>
+    </joint>
+    <link name="${robot_name}_link_ee">
+    </link>
+    <joint name="${robot_name}_joint_ee_kuka" type="fixed">
+      <parent link="${robot_name}_link_7"/>
       <child link="${robot_name}_link_ee_kuka"/>
       <origin xyz="0 0 0.045" rpy="${PI} ${PI} ${PI}"/>
@@ -299,11 +306,4 @@
     </joint>
     <link name="${robot_name}_link_ee_kuka">
-    </link>
-    <joint name="tool0_joint" type="fixed">
-      <parent link="${robot_name}_link_7"/>
-      <child link="${robot_name}_link_ee"/>
-      <origin xyz="0 0 0.045" rpy="0 -${PI/2} 0"/>
-    </joint>
-    <link name="${robot_name}_link_ee">
     </link>
     <!--Extensions -->

File: iiwa_description/urdf/iiwa7.urdf (robot description, URDF)
Before this commit: robot iiwa7, 11 links, 10 joints
Joints:
- removed joint tool0_joint
- added joint iiwa_joint_ee_kuka: type fixed, parent iiwa_link_7, child iiwa_link_ee_kuka, origin xyz=0 0 0.045 rpy=3.14159265359 3.14159265359 3.14159265359, axis 0 0 1
- joint iiwa_joint_ee: axis 0 0 1 -> (none); child iiwa_link_ee_kuka -> iiwa_link_ee; origin xyz=0 0 0.045 rpy=3.14159265359 3.14159265359 3.14159265359 -> xyz=0 0 0.045 rpy=0 -1.57079632679 0

File: iiwa_description/urdf/iiwa7.xacro (robot description, xacro)
@@ -22,27 +22,27 @@
     <link name="${robot_name}_link_0">
       <inertial>
-        <origin xyz="-0.1 0 0.07" rpy="0 0 0"/>
-        <mass value="5"/>
-        <inertia ixx="0.05"  ixy="0"  ixz="0" iyy="0.06" iyz="0" izz="0.03" />
-      </inertial>
-      <visual>
-        <origin xyz="0 0 0" rpy="0 0 0"/>
-        <geometry>
-          <mesh filename="package://iiwa_description/meshes/iiwa7/visual/link_0.stl"/>
-        </geometry>
-        <material name="Grey"/>
-      </visual>
-      <collision>
-        <origin xyz="0 0 0" rpy="0 0 0"/>
-        <geometry>
-          <mesh filename="package://iiwa_description/meshes/iiwa7/collision/link_0.stl"/>
-        </geometry>
-        <material name="Grey"/>
+	<origin xyz="-0.1 0 0.07" rpy="0 0 0"/>
+	<mass value="5"/>
+	<inertia ixx="0.05"  ixy="0"  ixz="0" iyy="0.06" iyz="0" izz="0.03" />
+      </inertial>
+      <visual>
+	<origin xyz="0 0 0" rpy="0 0 0"/>
+	<geometry>
+	  <mesh filename="package://iiwa_description/meshes/iiwa7/visual/link_0.stl"/>
+	</geometry>
+	<material name="Grey"/>
+      </visual>
+      <collision>
+	<origin xyz="0 0 0" rpy="0 0 0"/>
+	<geometry>
+	  <mesh filename="package://iiwa_description/meshes/iiwa7/collision/link_0.stl"/>
+	</geometry>
+	<material name="Grey"/>
       </collision>
       <self_collision_checking>
-        <origin xyz="0 0 0" rpy="0 0 0"/>
-        <geometry>
-          <capsule radius="0.15" length="0.25"/>
-        </geometry>
+	<origin xyz="0 0 0" rpy="0 0 0"/>
+	<geometry>
+	  <capsule radius="0.15" length="0.25"/>
+	</geometry>
       </self_collision_checking>
     </link>
@@ -54,30 +54,30 @@
       <axis xyz="0 0 1"/>
       <limit lower="${-170 * PI / 180}" upper="${170 * PI / 180}"
-             effort="${max_effort}" velocity="${max_velocity}" />
-         <safety_controller soft_lower_limit="${-168 * PI / 180}"
-           soft_upper_limit="${168 * PI / 180}"
-           k_position="${safety_controller_k_pos}"
-           k_velocity="${safety_controller_k_vel}"/>
+	     effort="${max_effort}" velocity="${max_velocity}" />
+      <safety_controller soft_lower_limit="${-168 * PI / 180}"
+			 soft_upper_limit="${168 * PI / 180}"
+			 k_position="${safety_controller_k_pos}"
+			 k_velocity="${safety_controller_k_vel}"/>
       <dynamics damping="${joint_damping}"/>
     </joint>
     <link name="${robot_name}_link_1">
       <inertial>
-        <origin xyz="0 -0.03 0.12" rpy="0 0 0"/>
-        <mass value="4"/>
-        <inertia ixx="0.1"  ixy="0"  ixz="0" iyy="0.09" iyz="0" izz="0.02" />
-      </inertial>
-      <visual>
-        <origin xyz="0 0 0.0075" rpy="0 0 0"/>
-        <geometry>
-          <mesh filename="package://iiwa_description/meshes/iiwa7/visual/link_1.stl"/>
-        </geometry>
-        <material name="Orange"/>
-      </visual>
-      <collision>
-        <origin xyz="0 0 0.0075" rpy="0 0 0"/>
-        <geometry>
-          <mesh filename="package://iiwa_description/meshes/iiwa7/collision/link_1.stl"/>
-        </geometry>
-        <material name="Orange"/>
+	<origin xyz="0 -0.03 0.12" rpy="0 0 0"/>
+	<mass value="4"/>
+	<inertia ixx="0.1"  ixy="0"  ixz="0" iyy="0.09" iyz="0" izz="0.02" />
+      </inertial>
+      <visual>
+	<origin xyz="0 0 0.0075" rpy="0 0 0"/>
+	<geometry>
+	  <mesh filename="package://iiwa_description/meshes/iiwa7/visual/link_1.stl"/>
+	</geometry>
+	<material name="Orange"/>
+      </visual>
+      <collision>
+	<origin xyz="0 0 0.0075" rpy="0 0 0"/>
+	<geometry>
+	  <mesh filename="package://iiwa_description/meshes/iiwa7/collision/link_1.stl"/>
+	</geometry>
+	<material name="Orange"/>
       </collision>
     </link>
@@ -88,30 +88,30 @@
       <axis xyz="0 0 1"/>
       <limit lower="${-120 * PI / 180}" upper="${120 * PI / 180}"
-             effort="${max_effort}" velocity="${max_velocity}" />
-       <safety_controller soft_lower_limit="${-118 * PI / 180}"
-           soft_upper_limit="${118 * PI / 180}"
-           k_position="${safety_controller_k_pos}"
-           k_velocity="${safety_controller_k_vel}"/>
+	     effort="${max_effort}" velocity="${max_velocity}" />
+      <safety_controller soft_lower_limit="${-118 * PI / 180}"
+			 soft_upper_limit="${118 * PI / 180}"
+			 k_position="${safety_controller_k_pos}"
+			 k_velocity="${safety_controller_k_vel}"/>
       <dynamics damping="${joint_damping}"/>
     </joint>
     <link name="${robot_name}_link_2">
       <inertial>
-        <origin xyz="0.0003 0.059 0.042" rpy="0 0 0"/>
-        <mass value="4"/>
-        <inertia ixx="0.05"  ixy="0"  ixz="0" iyy="0.018" iyz="0" izz="0.044" />
-      </inertial>
-      <visual>
-        <origin xyz="0 0 -0.0060" rpy="0 0 0"/>
-        <geometry>
-          <mesh filename="package://iiwa_description/meshes/iiwa7/visual/link_2.stl"/>
-        </geometry>
-        <material name="Orange"/>
-      </visual>
-      <collision>
-        <origin xyz="0 0 -0.0060" rpy="0 0 0"/>
-        <geometry>
-          <mesh filename="package://iiwa_description/meshes/iiwa7/collision/link_2.stl"/>
-        </geometry>
-        <material name="Orange"/>
+	<origin xyz="0.0003 0.059 0.042" rpy="0 0 0"/>
+	<mass value="4"/>
+	<inertia ixx="0.05"  ixy="0"  ixz="0" iyy="0.018" iyz="0" izz="0.044" />
+      </inertial>
+      <visual>
+	<origin xyz="0 0 -0.0060" rpy="0 0 0"/>
+	<geometry>
+	  <mesh filename="package://iiwa_description/meshes/iiwa7/visual/link_2.stl"/>
+	</geometry>
+	<material name="Orange"/>
+      </visual>
+      <collision>
+	<origin xyz="0 0 -0.0060" rpy="0 0 0"/>
+	<geometry>
+	  <mesh filename="package://iiwa_description/meshes/iiwa7/collision/link_2.stl"/>
+	</geometry>
+	<material name="Orange"/>
       </collision>
     </link>
@@ -122,30 +122,30 @@
       <axis xyz="0 0 1"/>
       <limit lower="${-170 * PI / 180}" upper="${170 * PI / 180}"
-             effort="${max_effort}" velocity="${max_velocity}" />
-       <safety_controller soft_lower_limit="${-168 * PI / 180}"
-           soft_upper_limit="${168 * PI / 180}"
-           k_position="${safety_controller_k_pos}"
-           k_velocity="${safety_controller_k_vel}"/>
+	     effort="${max_effort}" velocity="${max_velocity}" />
+      <safety_controller soft_lower_limit="${-168 * PI / 180}"
+			 soft_upper_limit="${168 * PI / 180}"
+			 k_position="${safety_controller_k_pos}"
+			 k_velocity="${safety_controller_k_vel}"/>
       <dynamics damping="${joint_damping}"/>
     </joint>
     <link name="${robot_name}_link_3">
       <inertial>
-        <origin xyz="0 0.03 0.13" rpy="0 0 0"/>
-        <mass value="3"/>
-        <inertia ixx="0.08"  ixy="0"  ixz="0" iyy="0.075" iyz="0" izz="0.01" />
-      </inertial>
-      <visual>
-        <origin xyz="0 -0.005 -0.026" rpy="0 0 0"/>
-        <geometry>
-          <mesh filename="package://iiwa_description/meshes/iiwa7/visual/link_3.stl"/>
-        </geometry>
-        <material name="Orange"/>
-      </visual>
-      <collision>
-        <origin xyz="0 -0.005 -0.026" rpy="0 0 0"/>
-        <geometry>
-          <mesh filename="package://iiwa_description/meshes/iiwa7/collision/link_3.stl"/>
-        </geometry>
-        <material name="Orange"/>
+	<origin xyz="0 0.03 0.13" rpy="0 0 0"/>
+	<mass value="3"/>
+	<inertia ixx="0.08"  ixy="0"  ixz="0" iyy="0.075" iyz="0" izz="0.01" />
+      </inertial>
+      <visual>
+	<origin xyz="0 -0.005 -0.026" rpy="0 0 0"/>
+	<geometry>
+	  <mesh filename="package://iiwa_description/meshes/iiwa7/visual/link_3.stl"/>
+	</geometry>
+	<material name="Orange"/>
+      </visual>
+      <collision>
+	<origin xyz="0 -0.005 -0.026" rpy="0 0 0"/>
+	<geometry>
+	  <mesh filename="package://iiwa_description/meshes/iiwa7/collision/link_3.stl"/>
+	</geometry>
+	<material name="Orange"/>
       </collision>
     </link>
@@ -156,30 +156,30 @@
       <axis xyz="0 0 1"/>
       <limit lower="${-120 * PI / 180}" upper="${120 * PI / 180}"
-             effort="${max_effort}" velocity="${max_velocity}" />
-       <safety_controller soft_lower_limit="${-118 * PI / 180}"
-           soft_upper_limit="${118 * PI / 180}"
-           k_position="${safety_controller_k_pos}"
-           k_velocity="${safety_controller_k_vel}"/>
+	     effort="${max_effort}" velocity="${max_velocity}" />
+      <safety_controller soft_lower_limit="${-118 * PI / 180}"
+			 soft_upper_limit="${118 * PI / 180}"
+			 k_position="${safety_controller_k_pos}"
+			 k_velocity="${safety_controller_k_vel}"/>
       <dynamics damping="${joint_damping}"/>
     </joint>
     <link name="${robot_name}_link_4">
       <inertial>
-        <origin xyz="0 0.067 0.034" rpy="0 0 0"/>
-        <mass value="2.7"/>
-        <inertia ixx="0.03"  ixy="0"  ixz="0" iyy="0.01" iyz="0" izz="0.029" />
-      </inertial>
-      <visual>
-        <origin xyz="0 0 0" rpy="0 0 0"/>
-        <geometry>
-          <mesh filename="package://iiwa_description/meshes/iiwa7/visual/link_4.stl"/>
-        </geometry>
-        <material name="Orange"/>
-      </visual>
-      <collision>
-        <origin xyz="0 0 0" rpy="0 0 0"/>
-        <geometry>
-          <mesh filename="package://iiwa_description/meshes/iiwa7/collision/link_4.stl"/>
-        </geometry>
-        <material name="Orange"/>
+	<origin xyz="0 0.067 0.034" rpy="0 0 0"/>
+	<mass value="2.7"/>
+	<inertia ixx="0.03"  ixy="0"  ixz="0" iyy="0.01" iyz="0" izz="0.029" />
+      </inertial>
+      <visual>
+	<origin xyz="0 0 0" rpy="0 0 0"/>
+	<geometry>
+	  <mesh filename="package://iiwa_description/meshes/iiwa7/visual/link_4.stl"/>
+	</geometry>
+	<material name="Orange"/>
+      </visual>
+      <collision>
+	<origin xyz="0 0 0" rpy="0 0 0"/>
+	<geometry>
+	  <mesh filename="package://iiwa_description/meshes/iiwa7/collision/link_4.stl"/>
+	</geometry>
+	<material name="Orange"/>
       </collision>
     </link>
@@ -190,30 +190,30 @@
       <axis xyz="0 0 1"/>
       <limit lower="${-170 * PI / 180}" upper="${170 * PI / 180}"
-             effort="${max_effort}" velocity="${max_velocity}" />
-       <safety_controller soft_lower_limit="${-168 * PI / 180}"
-           soft_upper_limit="${168 * PI / 180}"
-           k_position="${safety_controller_k_pos}"
-           k_velocity="${safety_controller_k_vel}"/>
+	     effort="${max_effort}" velocity="${max_velocity}" />
+      <safety_controller soft_lower_limit="${-168 * PI / 180}"
+			 soft_upper_limit="${168 * PI / 180}"
+			 k_position="${safety_controller_k_pos}"
+			 k_velocity="${safety_controller_k_vel}"/>
       <dynamics damping="${joint_damping}"/>
     </joint>
     <link name="${robot_name}_link_5">
       <inertial>
-        <origin xyz="0.0001 0.021 0.076" rpy="0 0 0"/>
-        <mass value="1.7"/>
-        <inertia ixx="0.02"  ixy="0"  ixz="0" iyy="0.018" iyz="0" izz="0.005" />
-      </inertial>
-      <visual>
-        <origin xyz="0 0 -0.026" rpy="0 0 0"/>
-        <geometry>
-          <mesh filename="package://iiwa_description/meshes/iiwa7/visual/link_5.stl"/>
-        </geometry>
-        <material name="Orange"/>
-      </visual>
-      <collision>
-        <origin xyz="0 0 -0.026" rpy="0 0 0"/>
-        <geometry>
-          <mesh filename="package://iiwa_description/meshes/iiwa7/collision/link_5.stl"/>
-        </geometry>
-        <material name="Orange"/>
+	<origin xyz="0.0001 0.021 0.076" rpy="0 0 0"/>
+	<mass value="1.7"/>
+	<inertia ixx="0.02"  ixy="0"  ixz="0" iyy="0.018" iyz="0" izz="0.005" />
+      </inertial>
+      <visual>
+	<origin xyz="0 0 -0.026" rpy="0 0 0"/>
+	<geometry>
+	  <mesh filename="package://iiwa_description/meshes/iiwa7/visual/link_5.stl"/>
+	</geometry>
+	<material name="Orange"/>
+      </visual>
+      <collision>
+	<origin xyz="0 0 -0.026" rpy="0 0 0"/>
+	<geometry>
+	  <mesh filename="package://iiwa_description/meshes/iiwa7/collision/link_5.stl"/>
+	</geometry>
+	<material name="Orange"/>
       </collision>
     </link>
@@ -224,30 +224,30 @@
       <axis xyz="0 0 1"/>
       <limit lower="${-120 * PI / 180}" upper="${120 * PI / 180}"
-             effort="${max_effort}" velocity="${max_velocity}" />
-       <safety_controller soft_lower_limit="${-118 * PI / 180}"
-           soft_upper_limit="${118 * PI / 180}"
-           k_position="${safety_controller_k_pos}"
-           k_velocity="${safety_controller_k_vel}"/>
+	     effort="${max_effort}" velocity="${max_velocity}" />
+      <safety_controller soft_lower_limit="${-118 * PI / 180}"
+			 soft_upper_limit="${118 * PI / 180}"
+			 k_position="${safety_controller_k_pos}"
+			 k_velocity="${safety_controller_k_vel}"/>
       <dynamics damping="${joint_damping}"/>
     </joint>
     <link name="${robot_name}_link_6">
       <inertial>
-        <origin xyz="0 0.0006 0.0004" rpy="0 0 0"/>
-        <mass value="1.8"/>
-        <inertia ixx="0.005"  ixy="0"  ixz="0" iyy="0.0036" iyz="0" izz="0.0047" />
-      </inertial>
-      <visual>
-        <origin xyz="0 0 0" rpy="0 0 0"/>
-        <geometry>
-          <mesh filename="package://iiwa_description/meshes/iiwa7/visual/link_6.stl"/>
-        </geometry>
-        <material name="Orange"/>
-      </visual>
-      <collision>
-        <origin xyz="0 0 0" rpy="0 0 0"/>
-        <geometry>
-          <mesh filename="package://iiwa_description/meshes/iiwa7/collision/link_6.stl"/>
-        </geometry>
-        <material name="Orange"/>
+	<origin xyz="0 0.0006 0.0004" rpy="0 0 0"/>
+	<mass value="1.8"/>
+	<inertia ixx="0.005"  ixy="0"  ixz="0" iyy="0.0036" iyz="0" izz="0.0047" />
+      </inertial>
+      <visual>
+	<origin xyz="0 0 0" rpy="0 0 0"/>
+	<geometry>
+	  <mesh filename="package://iiwa_description/meshes/iiwa7/visual/link_6.stl"/>
+	</geometry>
+	<material name="Orange"/>
+      </visual>
+      <collision>
+	<origin xyz="0 0 0" rpy="0 0 0"/>
+	<geometry>
+	  <mesh filename="package://iiwa_description/meshes/iiwa7/collision/link_6.stl"/>
+	</geometry>
+	<material name="Orange"/>
       </collision>
     </link>
@@ -258,33 +258,40 @@
       <axis xyz="0 0 1"/>
       <limit lower="${-175 * PI / 180}" upper="${175 * PI / 180}"
-             effort="${max_effort}" velocity="${max_velocity}" />
-       <safety_controller soft_lower_limit="${-173 * PI / 180}"
-           soft_upper_limit="${173 * PI / 180}"
-           k_position="${safety_controller_k_pos}"
-           k_velocity="${safety_controller_k_vel}"/>
+	     effort="${max_effort}" velocity="${max_velocity}" />
+      <safety_controller soft_lower_limit="${-173 * PI / 180}"
+			 soft_upper_limit="${173 * PI / 180}"
+			 k_position="${safety_controller_k_pos}"
+			 k_velocity="${safety_controller_k_vel}"/>
       <dynamics damping="${joint_damping}"/>
     </joint>
     <link name="${robot_name}_link_7">
       <inertial>
-        <origin xyz="0 0 0.02" rpy="0 0 0"/>
-        <mass value="0.3"/>
-        <inertia ixx="0.001"  ixy="0"  ixz="0" iyy="0.001" iyz="0" izz="0.001" />
-      </inertial>
-      <visual>
-        <origin xyz="0 0 -0.0005" rpy="0 0 0"/>
-        <geometry>
-          <mesh filename="package://iiwa_description/meshes/iiwa7/visual/link_7_basic.stl"/>
-        </geometry>
-        <material name="Grey"/>
-      </visual>
-      <collision>
-        <origin xyz="0 0 -0.0005" rpy="0 0 0"/>
-        <geometry>
-          <mesh filename="package://iiwa_description/meshes/iiwa7/collision/link_7_basic.stl"/>
-        </geometry>
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