Commit message: small tuning
Former-commit-id: fc0ba504061122f28aca4d31f9bc81e2ef19d39f

File: iiwa_description/urdf/iiwa7.xacro (robot description, xacro)
@@ -85,5 +85,5 @@
       <parent link="iiwa_link_1"/>
       <child link="iiwa_link_2"/>
-      <origin xyz="0 -0.0005 0.1840" rpy="${PI / 2}   0 ${PI}"/>
+      <origin xyz="0 0 0.1840" rpy="${PI / 2}   0 ${PI}"/>
       <axis xyz="0 0 1"/>
       <limit lower="${-120 * PI / 180}" upper="${120 * PI / 180}"
@@ -255,5 +255,5 @@
       <parent link="iiwa_link_6"/>
       <child link="iiwa_link_7"/>
-      <origin xyz="0 0.0805 0.060" rpy="${- PI / 2} ${PI} 0"/>
+      <origin xyz="0 0.0805 0.06070" rpy="${- PI / 2} ${PI} 0"/>
       <axis xyz="0 0 1"/>
       <limit lower="${-175 * PI / 180}" upper="${175 * PI / 180}"

Commit message: URDF is perfect wrt to end effector position. Link 3 doesn't look that nice when the robot rotates around joint 2, I believe it's kuka's fault.
Former-commit-id: b1980fc2b7fe80fa53fb4dc97e657153098913ee

File: iiwa_description/urdf/iiwa7.xacro (robot description, xacro)
@@ -51,5 +51,5 @@
       <parent link="iiwa_link_0"/>
       <child link="iiwa_link_1"/>
-      <origin xyz="0 0 0.1575" rpy="0 0 0"/>
+      <origin xyz="0 0 0.15" rpy="0 0 0"/>
       <axis xyz="0 0 1"/>
       <limit lower="${-170 * PI / 180}" upper="${170 * PI / 180}"
@@ -68,5 +68,5 @@
       </inertial>
       <visual>
-        <origin xyz="0 0 0" rpy="0 0 0"/>
+        <origin xyz="0 0 0.0075" rpy="0 0 0"/>
         <geometry>
           <mesh filename="package://iiwa_description/meshes/iiwa7/visual/link_1.stl"/>
@@ -75,5 +75,5 @@
       </visual>
       <collision>
-        <origin xyz="0 0 0" rpy="0 0 0"/>
+        <origin xyz="0 0 0.0075" rpy="0 0 0"/>
         <geometry>
           <mesh filename="package://iiwa_description/meshes/iiwa7/collision/link_1.stl"/>
@@ -85,5 +85,5 @@
       <parent link="iiwa_link_1"/>
       <child link="iiwa_link_2"/>
-      <origin xyz="0 0 0.1840" rpy="${PI / 2}   0 ${PI}"/>
+      <origin xyz="0 0 0.19" rpy="${PI / 2}   0 ${PI}"/>
       <axis xyz="0 0 1"/>
       <limit lower="${-120 * PI / 180}" upper="${120 * PI / 180}"
@@ -102,5 +102,5 @@
       </inertial>
       <visual>
-        <origin xyz="0 0 0" rpy="0 0 0"/>
+        <origin xyz="0 0 -0.0060" rpy="0 0 0"/>
         <geometry>
           <mesh filename="package://iiwa_description/meshes/iiwa7/visual/link_2.stl"/>
@@ -109,5 +109,5 @@
       </visual>
       <collision>
-        <origin xyz="0 0 0" rpy="0 0 0"/>
+        <origin xyz="0 0 -0.0060" rpy="0 0 0"/>
         <geometry>
           <mesh filename="package://iiwa_description/meshes/iiwa7/collision/link_2.stl"/>
@@ -119,5 +119,5 @@
       <parent link="iiwa_link_2"/>
       <child link="iiwa_link_3"/>
-      <origin xyz="0 0.184 0" rpy="${PI / 2} 0 ${PI}"/>
+      <origin xyz="0 0.21 0" rpy="${PI / 2} 0 ${PI}"/>
       <axis xyz="0 0 1"/>
       <limit lower="${-170 * PI / 180}" upper="${170 * PI / 180}"
@@ -136,5 +136,5 @@
       </inertial>
       <visual>
-        <origin xyz="0 0 0" rpy="0 0 0"/>
+        <origin xyz="0 -0.005 -0.026" rpy="0 0 0"/>
         <geometry>
           <mesh filename="package://iiwa_description/meshes/iiwa7/visual/link_3.stl"/>
@@ -143,5 +143,5 @@
       </visual>
       <collision>
-        <origin xyz="0 0 0" rpy="0 0 0"/>
+        <origin xyz="0 -0.005 -0.026" rpy="0 0 0"/>
         <geometry>
           <mesh filename="package://iiwa_description/meshes/iiwa7/collision/link_3.stl"/>
@@ -153,5 +153,5 @@
       <parent link="iiwa_link_3"/>
       <child link="iiwa_link_4"/>
-      <origin xyz="0 0 0.21550" rpy="${PI / 2} 0 0"/>
+      <origin xyz="0 0 0.19" rpy="${PI / 2} 0 0"/>
       <axis xyz="0 0 1"/>
       <limit lower="${-120 * PI / 180}" upper="${120 * PI / 180}"
@@ -187,5 +187,5 @@
       <parent link="iiwa_link_4"/>
       <child link="iiwa_link_5"/>-169
-      <origin xyz="0 0.1840 0" rpy="${-PI / 2} ${PI} 0"/>
+      <origin xyz="0 0.21 0" rpy="${-PI / 2} ${PI} 0"/>
       <axis xyz="0 0 1"/>
       <limit lower="${-175 * PI / 180}" upper="${175 * PI / 180}"
@@ -204,5 +204,5 @@
       </inertial>
       <visual>
-        <origin xyz="0 0 0" rpy="0 0 0"/>
+        <origin xyz="0 0 -0.026" rpy="0 0 0"/>
         <geometry>
           <mesh filename="package://iiwa_description/meshes/iiwa7/visual/link_5.stl"/>
@@ -211,5 +211,5 @@
       </visual>
       <collision>
-        <origin xyz="0 0 0" rpy="0 0 0"/>
+        <origin xyz="0 0 -0.026" rpy="0 0 0"/>
         <geometry>
           <mesh filename="package://iiwa_description/meshes/iiwa7/collision/link_5.stl"/>
@@ -221,5 +221,5 @@
       <parent link="iiwa_link_5"/>
       <child link="iiwa_link_6"/>
-      <origin xyz="0 0.06070 0.21550" rpy="${PI / 2} 0 0"/>
+      <origin xyz="0 0.06070 0.19" rpy="${PI / 2} 0 0"/>
       <axis xyz="0 0 1"/>
       <limit lower="${-120 * PI / 180}" upper="${120 * PI / 180}"
@@ -255,5 +255,5 @@
       <parent link="iiwa_link_6"/>
       <child link="iiwa_link_7"/>
-      <origin xyz="0 0.0805 0.06070" rpy="${- PI / 2} ${PI} 0"/>
+      <origin xyz="0 0.081 0.06070" rpy="${- PI / 2} ${PI} 0"/>
       <axis xyz="0 0 1"/>
       <limit lower="${-175 * PI / 180}" upper="${175 * PI / 180}"
@@ -272,5 +272,5 @@
       </inertial>
       <visual>
-        <origin xyz="0 0 0" rpy="0 0 0"/>
+        <origin xyz="0 0 -0.0005" rpy="0 0 0"/>
         <geometry>
           <mesh filename="package://iiwa_description/meshes/iiwa7/visual/link_7_basic.stl"/>
@@ -279,5 +279,5 @@
       </visual>
       <collision>
-        <origin xyz="0 0 0" rpy="0 0 0"/>
+        <origin xyz="0 0 -0.0005" rpy="0 0 0"/>
         <geometry>
           <mesh filename="package://iiwa_description/meshes/iiwa7/collision/link_7_basic.stl"/>

Commit message: Added intertia values from paper to the urdf file

File: iiwa_description/urdf/iiwa7.xacro (robot description, xacro)
@@ -64,6 +64,6 @@
       <inertial>
 	<origin xyz="0 -0.03 0.12" rpy="0 0 0"/>
-	<mass value="4"/>
-	<inertia ixx="0.1"  ixy="0"  ixz="0" iyy="0.09" iyz="0" izz="0.02" />
+	<mass value="3.4525"/>
+	<inertia ixx="0.02183"  ixy="0"  ixz="0" iyy="0.007703" iyz="-0.003887" izz="0.02083" />
       </inertial>
       <visual>
@@ -98,6 +98,6 @@
       <inertial>
 	<origin xyz="0.0003 0.059 0.042" rpy="0 0 0"/>
-	<mass value="4"/>
-	<inertia ixx="0.05"  ixy="0"  ixz="0" iyy="0.018" iyz="0" izz="0.044" />
+	<mass value="3.4821"/>
+	<inertia ixx="0.02076"  ixy="0"  ixz="-0.003626" iyy="0.02179" iyz="0" izz="0.00779" />
       </inertial>
       <visual>
@@ -132,6 +132,6 @@
       <inertial>
 	<origin xyz="0 0.03 0.13" rpy="0 0 0"/>
-	<mass value="3"/>
-	<inertia ixx="0.08"  ixy="0"  ixz="0" iyy="0.075" iyz="0" izz="0.01" />
+	<mass value="4.05623"/>
+	<inertia ixx="0.03204"  ixy="0"  ixz="0" iyy="0.00972" iyz="0.006227" izz="0.03042" />
       </inertial>
       <visual>
@@ -166,6 +166,6 @@
       <inertial>
 	<origin xyz="0 0.067 0.034" rpy="0 0 0"/>
-	<mass value="2.7"/>
-	<inertia ixx="0.03"  ixy="0"  ixz="0" iyy="0.01" iyz="0" izz="0.029" />
+	<mass value="3.4822"/>
+	<inertia ixx="0.02178"  ixy="0"  ixz="0" iyy="0.02075" iyz="-0.003625" izz="0.007785" />
       </inertial>
       <visual>
@@ -200,6 +200,6 @@
       <inertial>
 	<origin xyz="0.0001 0.021 0.076" rpy="0 0 0"/>
-	<mass value="1.7"/>
-	<inertia ixx="0.02"  ixy="0"  ixz="0" iyy="0.018" iyz="0" izz="0.005" />
+	<mass value="2.1633"/>
+	<inertia ixx="0.01287"  ixy="0"  ixz="0" iyy="0.005708" iyz="-0.003946" izz="0.01112" />
       </inertial>
       <visual>
@@ -234,6 +234,6 @@
       <inertial>
 	<origin xyz="0 0.0006 0.0004" rpy="0 0 0"/>
-	<mass value="1.8"/>
-	<inertia ixx="0.005"  ixy="0"  ixz="0" iyy="0.0036" iyz="0" izz="0.0047" />
+	<mass value="2.3466"/>
+	<inertia ixx="0.006509"  ixy="0"  ixz="0" iyy="0.006259" iyz="0.00031891" izz="0.004527" />
       </inertial>
       <visual>
@@ -268,6 +268,6 @@
       <inertial>
 	<origin xyz="0 0 0.02" rpy="0 0 0"/>
-	<mass value="0.3"/>
-	<inertia ixx="0.001"  ixy="0"  ixz="0" iyy="0.001" iyz="0" izz="0.001" />
+	<mass value="3.129"/>
+	<inertia ixx="0.01464"  ixy="0.0005912"  ixz="0" iyy="0.01465" iyz="0" izz="0.002872" />
       </inertial>
       <visual>

Commit message: reduced quality of the meshes This might help performance in rviz

File: iiwa_description/urdf/iiwa7.xacro (robot description, xacro)
@@ -274,5 +274,5 @@
 	<origin xyz="0 0 -0.0005" rpy="0 0 0"/>
 	<geometry>
-	  <mesh filename="package://iiwa_description/meshes/iiwa7/visual/link_7_basic.stl"/>
+	  <mesh filename="package://iiwa_description/meshes/iiwa7/visual/link_7.stl"/>
 	</geometry>
 	<material name="Grey"/>
@@ -281,5 +281,5 @@
 	<origin xyz="0 0 -0.0005" rpy="0 0 0"/>
 	<geometry>
-	  <mesh filename="package://iiwa_description/meshes/iiwa7/collision/link_7_basic.stl"/>
+	  <mesh filename="package://iiwa_description/meshes/iiwa7/collision/link_7.stl"/>
 	</geometry>
 	<material name="Grey"/>

Commit message: Changed iiwa7.xarco link2 and 3 transform to eliminate link misalignment.

File: iiwa_description/urdf/iiwa7.xacro (robot description, xacro)
@@ -102,5 +102,5 @@
       </inertial>
       <visual>
-	<origin xyz="0 0 -0.0060" rpy="0 0 0"/>
+	<origin xyz="0 0 0" rpy="0 0 0"/>
 	<geometry>
 	  <mesh filename="package://iiwa_description/meshes/iiwa7/visual/link_2.stl"/>
@@ -109,5 +109,5 @@
       </visual>
       <collision>
-	<origin xyz="0 0 -0.0060" rpy="0 0 0"/>
+	<origin xyz="0 0 0" rpy="0 0 0"/>
 	<geometry>
 	  <mesh filename="package://iiwa_description/meshes/iiwa7/collision/link_2.stl"/>
@@ -136,5 +136,5 @@
       </inertial>
       <visual>
-	<origin xyz="0 -0.005 -0.026" rpy="0 0 0"/>
+	<origin xyz="0 0 -0.026" rpy="0 0 0"/>
 	<geometry>
 	  <mesh filename="package://iiwa_description/meshes/iiwa7/visual/link_3.stl"/>
@@ -143,5 +143,5 @@
       </visual>
       <collision>
-	<origin xyz="0 -0.005 -0.026" rpy="0 0 0"/>
+	<origin xyz="0 0 -0.026" rpy="0 0 0"/>
 	<geometry>
 	  <mesh filename="package://iiwa_description/meshes/iiwa7/collision/link_3.stl"/>
