Commit message: meshes for iiwa14 moved
Former-commit-id: 56e31a0254e3e71fa30156300bb448984d3d337a

File: iiwa_description/urdf/iiwa14.xacro (robot description, xacro)
@@ -29,5 +29,5 @@
         <origin xyz="0 0 0" rpy="0 0 0"/>
         <geometry>
-          <mesh filename="package://iiwa_description/meshes/link_0.stl"/>
+          <mesh filename="package://iiwa_description/meshes/iiwa14/visual/link_0.stl"/>
         </geometry>
         <material name="Grey"/>
@@ -36,5 +36,5 @@
         <origin xyz="0 0 0" rpy="0 0 0"/>
         <geometry>
-          <mesh filename="package://iiwa_description/meshes/coarse/link_0.stl"/>
+          <mesh filename="package://iiwa_description/meshes/iiwa14/collision/link_0.stl"/>
         </geometry>
         <material name="Grey"/>
@@ -70,12 +70,12 @@
         <origin xyz="0 0 0" rpy="0 0 0"/>
         <geometry>
-          <mesh filename="package://iiwa_description/meshes/link_1.stl"/>
-        </geometry>
-        <material name="Orange"/>
-      </visual>
-      <collision>
-        <origin xyz="0 0 0" rpy="0 0 0"/>
-        <geometry>
-          <mesh filename="package://iiwa_description/meshes/coarse/link_1.stl"/>
+          <mesh filename="package://iiwa_description/meshes/iiwa14/visual/link_1.stl"/>
+        </geometry>
+        <material name="Orange"/>
+      </visual>
+      <collision>
+        <origin xyz="0 0 0" rpy="0 0 0"/>
+        <geometry>
+          <mesh filename="package://iiwa_description/meshes/iiwa14/collision/link_1.stl"/>
         </geometry>
         <material name="Orange"/>
@@ -105,12 +105,12 @@
         <origin xyz="0 0 0" rpy="0 0 0"/>
         <geometry>
-          <mesh filename="package://iiwa_description/meshes/link_2.stl"/>
-        </geometry>
-        <material name="Orange"/>
-      </visual>
-      <collision>
-        <origin xyz="0 0 0" rpy="0 0 0"/>
-        <geometry>
-          <mesh filename="package://iiwa_description/meshes/coarse/link_2.stl"/>
+          <mesh filename="package://iiwa_description/meshes/iiwa14/visual/link_2.stl"/>
+        </geometry>
+        <material name="Orange"/>
+      </visual>
+      <collision>
+        <origin xyz="0 0 0" rpy="0 0 0"/>
+        <geometry>
+          <mesh filename="package://iiwa_description/meshes/iiwa14/collision/link_2.stl"/>
         </geometry>
         <material name="Orange"/>
@@ -140,12 +140,12 @@
         <origin xyz="0 0 0" rpy="0 0 0"/>
         <geometry>
-          <mesh filename="package://iiwa_description/meshes/link_3.stl"/>
-        </geometry>
-        <material name="Orange"/>
-      </visual>
-      <collision>
-        <origin xyz="0 0 0" rpy="0 0 0"/>
-        <geometry>
-          <mesh filename="package://iiwa_description/meshes/coarse/link_3.stl"/>
+          <mesh filename="package://iiwa_description/meshes/iiwa14/visual/link_3.stl"/>
+        </geometry>
+        <material name="Orange"/>
+      </visual>
+      <collision>
+        <origin xyz="0 0 0" rpy="0 0 0"/>
+        <geometry>
+          <mesh filename="package://iiwa_description/meshes/iiwa14/collision/link_3.stl"/>
         </geometry>
         <material name="Orange"/>
@@ -175,12 +175,12 @@
         <origin xyz="0 0 0" rpy="0 0 0"/>
         <geometry>
-          <mesh filename="package://iiwa_description/meshes/link_4.stl"/>
-        </geometry>
-        <material name="Orange"/>
-      </visual>
-      <collision>
-        <origin xyz="0 0 0" rpy="0 0 0"/>
-        <geometry>
-          <mesh filename="package://iiwa_description/meshes/coarse/link_4.stl"/>
+          <mesh filename="package://iiwa_description/meshes/iiwa14/visual/link_4.stl"/>
+        </geometry>
+        <material name="Orange"/>
+      </visual>
+      <collision>
+        <origin xyz="0 0 0" rpy="0 0 0"/>
+        <geometry>
+          <mesh filename="package://iiwa_description/meshes/iiwa14/collision/link_4.stl"/>
         </geometry>
         <material name="Orange"/>
@@ -210,12 +210,12 @@
         <origin xyz="0 0 0" rpy="0 0 0"/>
         <geometry>
-          <mesh filename="package://iiwa_description/meshes/link_5.stl"/>
-        </geometry>
-        <material name="Orange"/>
-      </visual>
-      <collision>
-        <origin xyz="0 0 0" rpy="0 0 0"/>
-        <geometry>
-          <mesh filename="package://iiwa_description/meshes/coarse/link_5.stl"/>
+          <mesh filename="package://iiwa_description/meshes/iiwa14/visual/link_5.stl"/>
+        </geometry>
+        <material name="Orange"/>
+      </visual>
+      <collision>
+        <origin xyz="0 0 0" rpy="0 0 0"/>
+        <geometry>
+          <mesh filename="package://iiwa_description/meshes/iiwa14/collision/link_5.stl"/>
         </geometry>
         <material name="Orange"/>
@@ -245,12 +245,12 @@
         <origin xyz="0 0 0" rpy="0 0 0"/>
         <geometry>
-          <mesh filename="package://iiwa_description/meshes/link_6.stl"/>
-        </geometry>
-        <material name="Orange"/>
-      </visual>
-      <collision>
-        <origin xyz="0 0 0" rpy="0 0 0"/>
-        <geometry>
-          <mesh filename="package://iiwa_description/meshes/coarse/link_6.stl"/>
+          <mesh filename="package://iiwa_description/meshes/iiwa14/visual/link_6.stl"/>
+        </geometry>
+        <material name="Orange"/>
+      </visual>
+      <collision>
+        <origin xyz="0 0 0" rpy="0 0 0"/>
+        <geometry>
+          <mesh filename="package://iiwa_description/meshes/iiwa14/collision/link_6.stl"/>
         </geometry>
         <material name="Orange"/>
@@ -280,5 +280,5 @@
         <origin xyz="0 0 0" rpy="0 0 0"/>
         <geometry>
-          <mesh filename="package://iiwa_description/meshes/link_7.stl"/>
+          <mesh filename="package://iiwa_description/meshes/iiwa14/visual/link_7.stl"/>
         </geometry>
         <material name="Grey"/>
@@ -287,5 +287,5 @@
         <origin xyz="0 0 0" rpy="0 0 0"/>
         <geometry>
-          <mesh filename="package://iiwa_description/meshes/coarse/link_7.stl"/>
+          <mesh filename="package://iiwa_description/meshes/iiwa14/collision/link_7.stl"/>
         </geometry>
         <material name="Grey"/>

Commit message: limits for joint 7 were wrong
Former-commit-id: 578cab26534a065a14d182130bc27e290d1dbb30

File: iiwa_description/urdf/iiwa14.xacro (robot description, xacro)
@@ -265,6 +265,6 @@
       <limit lower="${-175 * PI / 180}" upper="${175 * PI / 180}"
              effort="${max_effort}" velocity="${max_velocity}" />
-       <safety_controller soft_lower_limit="${-118 * PI / 180}"
-           soft_upper_limit="${118 * PI / 180}"
+       <safety_controller soft_lower_limit="${-173 * PI / 180}"
+           soft_upper_limit="${173 * PI / 180}"
            k_position="${safety_controller_k_pos}"
            k_velocity="${safety_controller_k_vel}"/>

File: iiwa_description/urdf/iiwa7.xacro (robot description, xacro)
@@ -186,11 +186,11 @@
     <joint name="iiwa_joint_5" type="revolute">
       <parent link="iiwa_link_4"/>
-      <child link="iiwa_link_5"/>
+      <child link="iiwa_link_5"/>-169
       <origin xyz="0 0.1840 0" rpy="${-PI / 2} ${PI} 0"/>
       <axis xyz="0 0 1"/>
-      <limit lower="${-170 * PI / 180}" upper="${170 * PI / 180}"
-             effort="${max_effort}" velocity="${max_velocity}" />
-       <safety_controller soft_lower_limit="${-118 * PI / 180}"
-           soft_upper_limit="${118 * PI / 180}"
+      <limit lower="${-175 * PI / 180}" upper="${175 * PI / 180}"
+             effort="${max_effort}" velocity="${max_velocity}" />
+       <safety_controller soft_lower_limit="${-173 * PI / 180}"
+           soft_upper_limit="${173 * PI / 180}"
            k_position="${safety_controller_k_pos}"
            k_velocity="${safety_controller_k_vel}"/>
@@ -259,6 +259,6 @@
       <limit lower="${-175 * PI / 180}" upper="${175 * PI / 180}"
              effort="${max_effort}" velocity="${max_velocity}" />
-       <safety_controller soft_lower_limit="${-118 * PI / 180}"
-           soft_upper_limit="${118 * PI / 180}"
+       <safety_controller soft_lower_limit="${-173 * PI / 180}"
+           soft_upper_limit="${173 * PI / 180}"
            k_position="${safety_controller_k_pos}"
            k_velocity="${safety_controller_k_vel}"/>

Commit message: Joint and link names are now prefixed with robot_name for dual-arm setup

File: iiwa_description/urdf/iiwa14.xacro (robot description, xacro)
@@ -15,10 +15,10 @@
   <xacro:macro name="iiwa14" params="parent hardware_interface robot_name *origin">
     <!--joint between {parent} and link_0-->
-    <joint name="${parent}_joint" type="fixed">
+    <joint name="${parent}_${robot_name}_joint" type="fixed">
       <insert_block name="origin"/>
       <parent link="${parent}"/>
-      <child link="iiwa_link_0"/>
-    </joint>
-    <link name="iiwa_link_0">
+      <child link="${robot_name}_link_0"/>
+    </joint>
+    <link name="${robot_name}_link_0">
       <inertial>
         <origin xyz="-0.1 0 0.07" rpy="0 0 0"/>
@@ -48,7 +48,7 @@
     </link>
     <!-- joint between link_0 and link_1 -->
-    <joint name="iiwa_joint_1" type="revolute">
-      <parent link="iiwa_link_0"/>
-      <child link="iiwa_link_1"/>
+    <joint name="${robot_name}_joint_1" type="revolute">
+      <parent link="${robot_name}_link_0"/>
+      <child link="${robot_name}_link_1"/>
       <origin xyz="0 0 0.1575" rpy="0 0 0"/>
       <axis xyz="0 0 1"/>
@@ -61,5 +61,5 @@
       <dynamics damping="${joint_damping}"/>
     </joint>
-    <link name="iiwa_link_1">
+    <link name="${robot_name}_link_1">
       <inertial>
         <origin xyz="0 -0.03 0.12" rpy="0 0 0"/>
@@ -83,7 +83,7 @@
     </link>
     <!-- joint between link_1 and link_2 -->
-    <joint name="iiwa_joint_2" type="revolute">
-      <parent link="iiwa_link_1"/>
-      <child link="iiwa_link_2"/>
+    <joint name="${robot_name}_joint_2" type="revolute">
+      <parent link="${robot_name}_link_1"/>
+      <child link="${robot_name}_link_2"/>
       <origin xyz="0 0 0.2025" rpy="${PI / 2}   0 ${PI}"/>
       <axis xyz="0 0 1"/>
@@ -96,5 +96,5 @@
       <dynamics damping="${joint_damping}"/>
     </joint>
-    <link name="iiwa_link_2">
+    <link name="${robot_name}_link_2">
       <inertial>
         <origin xyz="0.0003 0.059 0.042" rpy="0 0 0"/>
@@ -118,7 +118,7 @@
     </link>
     <!-- joint between link_2 and link_3 -->
-    <joint name="iiwa_joint_3" type="revolute">
-      <parent link="iiwa_link_2"/>
-      <child link="iiwa_link_3"/>
+    <joint name="${robot_name}_joint_3" type="revolute">
+      <parent link="${robot_name}_link_2"/>
+      <child link="${robot_name}_link_3"/>
       <origin xyz="0 0.2045 0" rpy="${PI / 2} 0 ${PI}"/>
       <axis xyz="0 0 1"/>
@@ -131,5 +131,5 @@
       <dynamics damping="${joint_damping}"/>
     </joint>
-    <link name="iiwa_link_3">
+    <link name="${robot_name}_link_3">
       <inertial>
         <origin xyz="0 0.03 0.13" rpy="0 0 0"/>
@@ -153,7 +153,7 @@
     </link>
    <!-- joint between link_3 and link_4 -->
-    <joint name="iiwa_joint_4" type="revolute">
-      <parent link="iiwa_link_3"/>
-      <child link="iiwa_link_4"/>
+    <joint name="${robot_name}_joint_4" type="revolute">
+      <parent link="${robot_name}_link_3"/>
+      <child link="${robot_name}_link_4"/>
       <origin xyz="0 0 0.2155" rpy="${PI / 2} 0 0"/>
       <axis xyz="0 0 1"/>
@@ -166,5 +166,5 @@
       <dynamics damping="${joint_damping}"/>
     </joint>
-    <link name="iiwa_link_4">
+    <link name="${robot_name}_link_4">
       <inertial>
         <origin xyz="0 0.067 0.034" rpy="0 0 0"/>
@@ -188,7 +188,7 @@
     </link>
     <!-- joint between link_4 and link_5 -->
-    <joint name="iiwa_joint_5" type="revolute">
-      <parent link="iiwa_link_4"/>
-      <child link="iiwa_link_5"/>
+    <joint name="${robot_name}_joint_5" type="revolute">
+      <parent link="${robot_name}_link_4"/>
+      <child link="${robot_name}_link_5"/>
       <origin xyz="0 0.1845 0" rpy="${-PI / 2} ${PI} 0"/>
       <axis xyz="0 0 1"/>
@@ -201,5 +201,5 @@
       <dynamics damping="${joint_damping}"/>
     </joint>
-    <link name="iiwa_link_5">
+    <link name="${robot_name}_link_5">
       <inertial>
         <origin xyz="0.0001 0.021 0.076" rpy="0 0 0"/>
@@ -223,7 +223,7 @@
     </link>
  <!-- joint between link_5 and link_6 -->
-    <joint name="iiwa_joint_6" type="revolute">
-      <parent link="iiwa_link_5"/>
-      <child link="iiwa_link_6"/>
+    <joint name="${robot_name}_joint_6" type="revolute">
+      <parent link="${robot_name}_link_5"/>
+      <child link="${robot_name}_link_6"/>
       <origin xyz="0 0 0.2155" rpy="${PI / 2} 0 0"/>
       <axis xyz="0 0 1"/>
@@ -236,5 +236,5 @@
       <dynamics damping="${joint_damping}"/>
     </joint>
-    <link name="iiwa_link_6">
+    <link name="${robot_name}_link_6">
       <inertial>
         <origin xyz="0 0.0006 0.0004" rpy="0 0 0"/>
@@ -258,7 +258,7 @@
     </link>
  <!-- joint between link_6 and link_7 -->
-    <joint name="iiwa_joint_7" type="revolute">
-      <parent link="iiwa_link_6"/>
-      <child link="iiwa_link_7"/>
+    <joint name="${robot_name}_joint_7" type="revolute">
+      <parent link="${robot_name}_link_6"/>
+      <child link="${robot_name}_link_7"/>
       <origin xyz="0 0.081 0" rpy="${- PI / 2} ${PI} 0"/>
       <axis xyz="0 0 1"/>
@@ -271,5 +271,5 @@
       <dynamics damping="${joint_damping}"/>
     </joint>
-    <link name="iiwa_link_7">
+    <link name="${robot_name}_link_7">
       <inertial>
         <origin xyz="0 0 0.02" rpy="0 0 0"/>
@@ -292,11 +292,11 @@
       </collision>
     </link>
-    <joint name="iiwa_joint_ee" type="fixed">
-      <parent link="iiwa_link_7"/>
-      <child link="iiwa_link_ee"/>
+    <joint name="${robot_name}_joint_ee" type="fixed">
+      <parent link="${robot_name}_link_7"/>
+      <child link="${robot_name}_link_ee"/>
       <origin xyz="0 0 0.045" rpy="${PI} ${PI} ${PI}"/>
       <axis xyz="0 0 1"/>
     </joint>
-    <link name="iiwa_link_ee">
+    <link name="${robot_name}_link_ee">
     </link>
     <!--Extensions -->

File: iiwa_description/urdf/iiwa7.xacro (robot description, xacro)
@@ -15,10 +15,10 @@
   <xacro:macro name="iiwa7" params="parent hardware_interface robot_name *origin">
     <!--joint between {parent} and link_0-->
-    <joint name="${parent}_joint" type="fixed">
+    <joint name="${parent}_${robot_name}_joint" type="fixed">
       <insert_block name="origin"/>
       <parent link="${parent}"/>
-      <child link="iiwa_link_0"/>
-    </joint>
-    <link name="iiwa_link_0">
+      <child link="${robot_name}_link_0"/>
+    </joint>
+    <link name="${robot_name}_link_0">
       <inertial>
         <origin xyz="-0.1 0 0.07" rpy="0 0 0"/>
@@ -48,7 +48,7 @@
     </link>
     <!-- joint between link_0 and link_1 -->
-    <joint name="iiwa_joint_1" type="revolute">
-      <parent link="iiwa_link_0"/>
-      <child link="iiwa_link_1"/>
+    <joint name="${robot_name}_joint_1" type="revolute">
+      <parent link="${robot_name}_link_0"/>
+      <child link="${robot_name}_link_1"/>
       <origin xyz="0 0 0.15" rpy="0 0 0"/>
       <axis xyz="0 0 1"/>
@@ -61,5 +61,5 @@
       <dynamics damping="${joint_damping}"/>
     </joint>
-    <link name="iiwa_link_1">
+    <link name="${robot_name}_link_1">
       <inertial>
         <origin xyz="0 -0.03 0.12" rpy="0 0 0"/>
@@ -82,7 +82,7 @@
       </collision>
     </link>
-    <joint name="iiwa_joint_2" type="revolute">
-      <parent link="iiwa_link_1"/>
-      <child link="iiwa_link_2"/>
+    <joint name="${robot_name}_joint_2" type="revolute">
+      <parent link="${robot_name}_link_1"/>
+      <child link="${robot_name}_link_2"/>
       <origin xyz="0 0 0.19" rpy="${PI / 2}   0 ${PI}"/>
       <axis xyz="0 0 1"/>
@@ -95,5 +95,5 @@
       <dynamics damping="${joint_damping}"/>
     </joint>
-    <link name="iiwa_link_2">
+    <link name="${robot_name}_link_2">
       <inertial>
         <origin xyz="0.0003 0.059 0.042" rpy="0 0 0"/>
@@ -116,7 +116,7 @@
       </collision>
     </link>
-    <joint name="iiwa_joint_3" type="revolute">
-      <parent link="iiwa_link_2"/>
-      <child link="iiwa_link_3"/>
+    <joint name="${robot_name}_joint_3" type="revolute">
+      <parent link="${robot_name}_link_2"/>
+      <child link="${robot_name}_link_3"/>
       <origin xyz="0 0.21 0" rpy="${PI / 2} 0 ${PI}"/>
       <axis xyz="0 0 1"/>
@@ -129,5 +129,5 @@
       <dynamics damping="${joint_damping}"/>
     </joint>
-    <link name="iiwa_link_3">
+    <link name="${robot_name}_link_3">
       <inertial>
         <origin xyz="0 0.03 0.13" rpy="0 0 0"/>
@@ -150,7 +150,7 @@
       </collision>
     </link>
-    <joint name="iiwa_joint_4" type="revolute">
-      <parent link="iiwa_link_3"/>
-      <child link="iiwa_link_4"/>
+    <joint name="${robot_name}_joint_4" type="revolute">
+      <parent link="${robot_name}_link_3"/>
+      <child link="${robot_name}_link_4"/>
       <origin xyz="0 0 0.19" rpy="${PI / 2} 0 0"/>
       <axis xyz="0 0 1"/>
@@ -163,5 +163,5 @@
       <dynamics damping="${joint_damping}"/>
     </joint>
-    <link name="iiwa_link_4">
+    <link name="${robot_name}_link_4">
       <inertial>
         <origin xyz="0 0.067 0.034" rpy="0 0 0"/>
@@ -184,7 +184,7 @@
       </collision>
     </link>
-    <joint name="iiwa_joint_5" type="revolute">
-      <parent link="iiwa_link_4"/>
-      <child link="iiwa_link_5"/>-169
+    <joint name="${robot_name}_joint_5" type="revolute">
+      <parent link="${robot_name}_link_4"/>
+      <child link="${robot_name}_link_5"/>-169
       <origin xyz="0 0.21 0" rpy="${-PI / 2} ${PI} 0"/>
       <axis xyz="0 0 1"/>
@@ -197,5 +197,5 @@
       <dynamics damping="${joint_damping}"/>
     </joint>
-    <link name="iiwa_link_5">
+    <link name="${robot_name}_link_5">
       <inertial>
         <origin xyz="0.0001 0.021 0.076" rpy="0 0 0"/>
@@ -218,7 +218,7 @@
       </collision>
     </link>
-    <joint name="iiwa_joint_6" type="revolute">
-      <parent link="iiwa_link_5"/>
-      <child link="iiwa_link_6"/>
+    <joint name="${robot_name}_joint_6" type="revolute">
+      <parent link="${robot_name}_link_5"/>
+      <child link="${robot_name}_link_6"/>
       <origin xyz="0 0.06070 0.19" rpy="${PI / 2} 0 0"/>
       <axis xyz="0 0 1"/>
@@ -231,5 +231,5 @@
       <dynamics damping="${joint_damping}"/>
     </joint>
-    <link name="iiwa_link_6">
+    <link name="${robot_name}_link_6">
       <inertial>
         <origin xyz="0 0.0006 0.0004" rpy="0 0 0"/>
@@ -252,7 +252,7 @@
       </collision>
     </link>
-    <joint name="iiwa_joint_7" type="revolute">
-      <parent link="iiwa_link_6"/>
-      <child link="iiwa_link_7"/>
+    <joint name="${robot_name}_joint_7" type="revolute">
+      <parent link="${robot_name}_link_6"/>
+      <child link="${robot_name}_link_7"/>
       <origin xyz="0 0.081 0.06070" rpy="${- PI / 2} ${PI} 0"/>
       <axis xyz="0 0 1"/>
@@ -265,5 +265,5 @@
       <dynamics damping="${joint_damping}"/>
     </joint>
-    <link name="iiwa_link_7">
+    <link name="${robot_name}_link_7">
       <inertial>
         <origin xyz="0 0 0.02" rpy="0 0 0"/>
@@ -286,11 +286,11 @@
       </collision>
     </link>
-    <joint name="iiwa_joint_ee" type="fixed">
-      <parent link="iiwa_link_7"/>
-      <child link="iiwa_link_ee"/>
+    <joint name="${robot_name}_joint_ee" type="fixed">
+      <parent link="${robot_name}_link_7"/>
+      <child link="${robot_name}_link_ee"/>
       <origin xyz="0 0 0.045" rpy="${PI} ${PI} ${PI}"/>
       <axis xyz="0 0 1"/>
     </joint>
-    <link name="iiwa_link_ee">
+    <link name="${robot_name}_link_ee">
     </link>
     <!--Extensions -->

Commit message: fixed joint limits

File: iiwa_description/urdf/iiwa14.xacro (robot description, xacro)
@@ -125,6 +125,6 @@
       <limit lower="${-170 * PI / 180}" upper="${170 * PI / 180}"
              effort="${max_effort}" velocity="${max_velocity}" />
-       <safety_controller soft_lower_limit="${-118 * PI / 180}"
-           soft_upper_limit="${118 * PI / 180}"
+       <safety_controller soft_lower_limit="${-168 * PI / 180}"
+           soft_upper_limit="${168 * PI / 180}"
            k_position="${safety_controller_k_pos}"
            k_velocity="${safety_controller_k_vel}"/>
@@ -195,6 +195,6 @@
       <limit lower="${-170 * PI / 180}" upper="${170 * PI / 180}"
              effort="${max_effort}" velocity="${max_velocity}" />
-       <safety_controller soft_lower_limit="${-118 * PI / 180}"
-           soft_upper_limit="${118 * PI / 180}"
+       <safety_controller soft_lower_limit="${-168 * PI / 180}"
+           soft_upper_limit="${168 * PI / 180}"
            k_position="${safety_controller_k_pos}"
            k_velocity="${safety_controller_k_vel}"/>

File: iiwa_description/urdf/iiwa7.urdf (robot description, URDF)
Before this commit: robot iiwa7, 11 links, 10 joints
Joints:
- joint iiwa_joint_5: limit lower=-3.05432619099 upper=3.05432619099 effort=300 velocity=10 -> lower=-2.96705972839 upper=2.96705972839 effort=300 velocity=10

File: iiwa_description/urdf/iiwa7.xacro (robot description, xacro)
@@ -123,6 +123,6 @@
       <limit lower="${-170 * PI / 180}" upper="${170 * PI / 180}"
              effort="${max_effort}" velocity="${max_velocity}" />
-       <safety_controller soft_lower_limit="${-118 * PI / 180}"
-           soft_upper_limit="${118 * PI / 180}"
+       <safety_controller soft_lower_limit="${-168 * PI / 180}"
+           soft_upper_limit="${168 * PI / 180}"
            k_position="${safety_controller_k_pos}"
            k_velocity="${safety_controller_k_vel}"/>
@@ -189,8 +189,8 @@
       <origin xyz="0 0.21 0" rpy="${-PI / 2} ${PI} 0"/>
       <axis xyz="0 0 1"/>
-      <limit lower="${-175 * PI / 180}" upper="${175 * PI / 180}"
-             effort="${max_effort}" velocity="${max_velocity}" />
-       <safety_controller soft_lower_limit="${-173 * PI / 180}"
-           soft_upper_limit="${173 * PI / 180}"
+      <limit lower="${-170 * PI / 180}" upper="${170 * PI / 180}"
+             effort="${max_effort}" velocity="${max_velocity}" />
+       <safety_controller soft_lower_limit="${-168 * PI / 180}"
+           soft_upper_limit="${168 * PI / 180}"
            k_position="${safety_controller_k_pos}"
            k_velocity="${safety_controller_k_vel}"/>
