Commit message: Remove the _kuka frame in the model, notreally meaningful the way it was

File: iiwa_description/urdf/iiwa14.xacro (robot description, xacro)
@@ -295,15 +295,7 @@
       <parent link="${robot_name}_link_7"/>
       <child link="${robot_name}_link_ee"/>
-      <origin xyz="0 0 0.045" rpy="0 -${PI/2} 0"/>
+      <origin xyz="0 0 0.045" rpy="0 0 0"/>
     </joint>
     <link name="${robot_name}_link_ee">
-    </link>
-    <joint name="${robot_name}_joint_ee_kuka" type="fixed">
-      <parent link="${robot_name}_link_7"/>
-      <child link="${robot_name}_link_ee_kuka"/>
-      <origin xyz="0 0 0.045" rpy="${PI} ${PI} ${PI}"/>
-      <axis xyz="0 0 1"/>
-    </joint>
-    <link name="${robot_name}_link_ee_kuka">
     </link>
     <!--Extensions -->

File: iiwa_description/urdf/iiwa7.xacro (robot description, xacro)
@@ -289,15 +289,7 @@
       <parent link="${robot_name}_link_7"/>
       <child link="${robot_name}_link_ee"/>
-      <origin xyz="0 0 0.045" rpy="0 -${PI/2} 0"/>
+      <origin xyz="0 0 0.045" rpy="0 0 0"/>
     </joint>
     <link name="${robot_name}_link_ee">
-    </link>
-    <joint name="${robot_name}_joint_ee_kuka" type="fixed">
-      <parent link="${robot_name}_link_7"/>
-      <child link="${robot_name}_link_ee_kuka"/>
-      <origin xyz="0 0 0.045" rpy="${PI} ${PI} ${PI}"/>
-      <axis xyz="0 0 1"/>
-    </joint>
-    <link name="${robot_name}_link_ee_kuka">
     </link>
     <!--Extensions -->
