Commit message: modified xacros to have a parametric origin for the model

File: iiwa_description/urdf/iiwa7.xacro (robot description, xacro)
@@ -22,27 +22,27 @@
     <link name="${robot_name}_link_0">
       <inertial>
-	<origin xyz="-0.1 0 0.07" rpy="0 0 0"/>
-	<mass value="5"/>
-	<inertia ixx="0.05"  ixy="0"  ixz="0" iyy="0.06" iyz="0" izz="0.03" />
-      </inertial>
-      <visual>
-	<origin xyz="0 0 0" rpy="0 0 0"/>
-	<geometry>
-	  <mesh filename="package://iiwa_description/meshes/iiwa7/visual/link_0.stl"/>
-	</geometry>
-	<material name="Grey"/>
-      </visual>
-      <collision>
-	<origin xyz="0 0 0" rpy="0 0 0"/>
-	<geometry>
-	  <mesh filename="package://iiwa_description/meshes/iiwa7/collision/link_0.stl"/>
-	</geometry>
-	<material name="Grey"/>
+        <origin xyz="-0.1 0 0.07" rpy="0 0 0"/>
+        <mass value="5"/>
+        <inertia ixx="0.05"  ixy="0"  ixz="0" iyy="0.06" iyz="0" izz="0.03" />
+      </inertial>
+      <visual>
+        <origin xyz="0 0 0" rpy="0 0 0"/>
+        <geometry>
+          <mesh filename="package://iiwa_description/meshes/iiwa7/visual/link_0.stl"/>
+        </geometry>
+        <material name="Grey"/>
+      </visual>
+      <collision>
+        <origin xyz="0 0 0" rpy="0 0 0"/>
+        <geometry>
+          <mesh filename="package://iiwa_description/meshes/iiwa7/collision/link_0.stl"/>
+        </geometry>
+        <material name="Grey"/>
       </collision>
       <self_collision_checking>
-	<origin xyz="0 0 0" rpy="0 0 0"/>
-	<geometry>
-	  <capsule radius="0.15" length="0.25"/>
-	</geometry>
+        <origin xyz="0 0 0" rpy="0 0 0"/>
+        <geometry>
+          <capsule radius="0.15" length="0.25"/>
+        </geometry>
       </self_collision_checking>
     </link>
@@ -54,30 +54,30 @@
       <axis xyz="0 0 1"/>
       <limit lower="${-170 * PI / 180}" upper="${170 * PI / 180}"
-	     effort="${max_effort}" velocity="${max_velocity}" />
+             effort="${max_effort}" velocity="${max_velocity}" />
       <safety_controller soft_lower_limit="${-168 * PI / 180}"
-			 soft_upper_limit="${168 * PI / 180}"
-			 k_position="${safety_controller_k_pos}"
-			 k_velocity="${safety_controller_k_vel}"/>
+                         soft_upper_limit="${168 * PI / 180}"
+                         k_position="${safety_controller_k_pos}"
+                         k_velocity="${safety_controller_k_vel}"/>
       <dynamics damping="${joint_damping}"/>
     </joint>
     <link name="${robot_name}_link_1">
       <inertial>
-	<origin xyz="0 -0.03 0.12" rpy="0 0 0"/>
-	<mass value="3.4525"/>
-	<inertia ixx="0.02183"  ixy="0"  ixz="0" iyy="0.007703" iyz="-0.003887" izz="0.02083" />
-      </inertial>
-      <visual>
-	<origin xyz="0 0 0.0075" rpy="0 0 0"/>
-	<geometry>
-	  <mesh filename="package://iiwa_description/meshes/iiwa7/visual/link_1.stl"/>
-	</geometry>
-	<material name="Orange"/>
-      </visual>
-      <collision>
-	<origin xyz="0 0 0.0075" rpy="0 0 0"/>
-	<geometry>
-	  <mesh filename="package://iiwa_description/meshes/iiwa7/collision/link_1.stl"/>
-	</geometry>
-	<material name="Orange"/>
+        <origin xyz="0 -0.03 0.12" rpy="0 0 0"/>
+        <mass value="3.4525"/>
+        <inertia ixx="0.02183"  ixy="0"  ixz="0" iyy="0.007703" iyz="-0.003887" izz="0.02083" />
+      </inertial>
+      <visual>
+        <origin xyz="0 0 0.0075" rpy="0 0 0"/>
+        <geometry>
+          <mesh filename="package://iiwa_description/meshes/iiwa7/visual/link_1.stl"/>
+        </geometry>
+        <material name="Orange"/>
+      </visual>
+      <collision>
+        <origin xyz="0 0 0.0075" rpy="0 0 0"/>
+        <geometry>
+          <mesh filename="package://iiwa_description/meshes/iiwa7/collision/link_1.stl"/>
+        </geometry>
+        <material name="Orange"/>
       </collision>
     </link>
@@ -88,30 +88,30 @@
       <axis xyz="0 0 1"/>
       <limit lower="${-120 * PI / 180}" upper="${120 * PI / 180}"
-	     effort="${max_effort}" velocity="${max_velocity}" />
+             effort="${max_effort}" velocity="${max_velocity}" />
       <safety_controller soft_lower_limit="${-118 * PI / 180}"
-			 soft_upper_limit="${118 * PI / 180}"
-			 k_position="${safety_controller_k_pos}"
-			 k_velocity="${safety_controller_k_vel}"/>
+                         soft_upper_limit="${118 * PI / 180}"
+                         k_position="${safety_controller_k_pos}"
+                         k_velocity="${safety_controller_k_vel}"/>
       <dynamics damping="${joint_damping}"/>
     </joint>
     <link name="${robot_name}_link_2">
       <inertial>
-	<origin xyz="0.0003 0.059 0.042" rpy="0 0 0"/>
-	<mass value="3.4821"/>
-	<inertia ixx="0.02076"  ixy="0"  ixz="-0.003626" iyy="0.02179" iyz="0" izz="0.00779" />
-      </inertial>
-      <visual>
-	<origin xyz="0 0 0" rpy="0 0 0"/>
-	<geometry>
-	  <mesh filename="package://iiwa_description/meshes/iiwa7/visual/link_2.stl"/>
-	</geometry>
-	<material name="Orange"/>
-      </visual>
-      <collision>
-	<origin xyz="0 0 0" rpy="0 0 0"/>
-	<geometry>
-	  <mesh filename="package://iiwa_description/meshes/iiwa7/collision/link_2.stl"/>
-	</geometry>
-	<material name="Orange"/>
+        <origin xyz="0.0003 0.059 0.042" rpy="0 0 0"/>
+        <mass value="3.4821"/>
+        <inertia ixx="0.02076"  ixy="0"  ixz="-0.003626" iyy="0.02179" iyz="0" izz="0.00779" />
+      </inertial>
+      <visual>
+        <origin xyz="0 0 0" rpy="0 0 0"/>
+        <geometry>
+          <mesh filename="package://iiwa_description/meshes/iiwa7/visual/link_2.stl"/>
+        </geometry>
+        <material name="Orange"/>
+      </visual>
+      <collision>
+        <origin xyz="0 0 0" rpy="0 0 0"/>
+        <geometry>
+          <mesh filename="package://iiwa_description/meshes/iiwa7/collision/link_2.stl"/>
+        </geometry>
+        <material name="Orange"/>
       </collision>
     </link>
@@ -122,30 +122,30 @@
       <axis xyz="0 0 1"/>
       <limit lower="${-170 * PI / 180}" upper="${170 * PI / 180}"
-	     effort="${max_effort}" velocity="${max_velocity}" />
+             effort="${max_effort}" velocity="${max_velocity}" />
       <safety_controller soft_lower_limit="${-168 * PI / 180}"
-			 soft_upper_limit="${168 * PI / 180}"
-			 k_position="${safety_controller_k_pos}"
-			 k_velocity="${safety_controller_k_vel}"/>
+                         soft_upper_limit="${168 * PI / 180}"
+                         k_position="${safety_controller_k_pos}"
+                         k_velocity="${safety_controller_k_vel}"/>
       <dynamics damping="${joint_damping}"/>
     </joint>
     <link name="${robot_name}_link_3">
       <inertial>
-	<origin xyz="0 0.03 0.13" rpy="0 0 0"/>
-	<mass value="4.05623"/>
-	<inertia ixx="0.03204"  ixy="0"  ixz="0" iyy="0.00972" iyz="0.006227" izz="0.03042" />
-      </inertial>
-      <visual>
-	<origin xyz="0 0 -0.026" rpy="0 0 0"/>
-	<geometry>
-	  <mesh filename="package://iiwa_description/meshes/iiwa7/visual/link_3.stl"/>
-	</geometry>
-	<material name="Orange"/>
-      </visual>
-      <collision>
-	<origin xyz="0 0 -0.026" rpy="0 0 0"/>
-	<geometry>
-	  <mesh filename="package://iiwa_description/meshes/iiwa7/collision/link_3.stl"/>
-	</geometry>
-	<material name="Orange"/>
+        <origin xyz="0 0.03 0.13" rpy="0 0 0"/>
+        <mass value="4.05623"/>
+        <inertia ixx="0.03204"  ixy="0"  ixz="0" iyy="0.00972" iyz="0.006227" izz="0.03042" />
+      </inertial>
+      <visual>
+        <origin xyz="0 0 -0.026" rpy="0 0 0"/>
+        <geometry>
+          <mesh filename="package://iiwa_description/meshes/iiwa7/visual/link_3.stl"/>
+        </geometry>
+        <material name="Orange"/>
+      </visual>
+      <collision>
+        <origin xyz="0 0 -0.026" rpy="0 0 0"/>
+        <geometry>
+          <mesh filename="package://iiwa_description/meshes/iiwa7/collision/link_3.stl"/>
+        </geometry>
+        <material name="Orange"/>
       </collision>
     </link>
@@ -156,30 +156,30 @@
       <axis xyz="0 0 1"/>
       <limit lower="${-120 * PI / 180}" upper="${120 * PI / 180}"
-	     effort="${max_effort}" velocity="${max_velocity}" />
+             effort="${max_effort}" velocity="${max_velocity}" />
       <safety_controller soft_lower_limit="${-118 * PI / 180}"
-			 soft_upper_limit="${118 * PI / 180}"
-			 k_position="${safety_controller_k_pos}"
-			 k_velocity="${safety_controller_k_vel}"/>
+                         soft_upper_limit="${118 * PI / 180}"
+                         k_position="${safety_controller_k_pos}"
+                         k_velocity="${safety_controller_k_vel}"/>
       <dynamics damping="${joint_damping}"/>
     </joint>
     <link name="${robot_name}_link_4">
       <inertial>
-	<origin xyz="0 0.067 0.034" rpy="0 0 0"/>
-	<mass value="3.4822"/>
-	<inertia ixx="0.02178"  ixy="0"  ixz="0" iyy="0.02075" iyz="-0.003625" izz="0.007785" />
-      </inertial>
-      <visual>
-	<origin xyz="0 0 0" rpy="0 0 0"/>
-	<geometry>
-	  <mesh filename="package://iiwa_description/meshes/iiwa7/visual/link_4.stl"/>
-	</geometry>
-	<material name="Orange"/>
-      </visual>
-      <collision>
-	<origin xyz="0 0 0" rpy="0 0 0"/>
-	<geometry>
-	  <mesh filename="package://iiwa_description/meshes/iiwa7/collision/link_4.stl"/>
-	</geometry>
-	<material name="Orange"/>
+        <origin xyz="0 0.067 0.034" rpy="0 0 0"/>
+        <mass value="3.4822"/>
+        <inertia ixx="0.02178"  ixy="0"  ixz="0" iyy="0.02075" iyz="-0.003625" izz="0.007785" />
+      </inertial>
+      <visual>
+        <origin xyz="0 0 0" rpy="0 0 0"/>
+        <geometry>
+          <mesh filename="package://iiwa_description/meshes/iiwa7/visual/link_4.stl"/>
+        </geometry>
+        <material name="Orange"/>
+      </visual>
+      <collision>
+        <origin xyz="0 0 0" rpy="0 0 0"/>
+        <geometry>
+          <mesh filename="package://iiwa_description/meshes/iiwa7/collision/link_4.stl"/>
+        </geometry>
+        <material name="Orange"/>
       </collision>
     </link>
@@ -190,30 +190,30 @@
       <axis xyz="0 0 1"/>
       <limit lower="${-170 * PI / 180}" upper="${170 * PI / 180}"
-	     effort="${max_effort}" velocity="${max_velocity}" />
+             effort="${max_effort}" velocity="${max_velocity}" />
       <safety_controller soft_lower_limit="${-168 * PI / 180}"
-			 soft_upper_limit="${168 * PI / 180}"
-			 k_position="${safety_controller_k_pos}"
-			 k_velocity="${safety_controller_k_vel}"/>
+                         soft_upper_limit="${168 * PI / 180}"
+                         k_position="${safety_controller_k_pos}"
+                         k_velocity="${safety_controller_k_vel}"/>
       <dynamics damping="${joint_damping}"/>
     </joint>
     <link name="${robot_name}_link_5">
       <inertial>
-	<origin xyz="0.0001 0.021 0.076" rpy="0 0 0"/>
-	<mass value="2.1633"/>
-	<inertia ixx="0.01287"  ixy="0"  ixz="0" iyy="0.005708" iyz="-0.003946" izz="0.01112" />
-      </inertial>
-      <visual>
-	<origin xyz="0 0 -0.026" rpy="0 0 0"/>
-	<geometry>
-	  <mesh filename="package://iiwa_description/meshes/iiwa7/visual/link_5.stl"/>
-	</geometry>
-	<material name="Orange"/>
-      </visual>
-      <collision>
-	<origin xyz="0 0 -0.026" rpy="0 0 0"/>
-	<geometry>
-	  <mesh filename="package://iiwa_description/meshes/iiwa7/collision/link_5.stl"/>
-	</geometry>
-	<material name="Orange"/>
+        <origin xyz="0.0001 0.021 0.076" rpy="0 0 0"/>
+        <mass value="2.1633"/>
+        <inertia ixx="0.01287"  ixy="0"  ixz="0" iyy="0.005708" iyz="-0.003946" izz="0.01112" />
+      </inertial>
+      <visual>
+        <origin xyz="0 0 -0.026" rpy="0 0 0"/>
+        <geometry>
+          <mesh filename="package://iiwa_description/meshes/iiwa7/visual/link_5.stl"/>
+        </geometry>
+        <material name="Orange"/>
+      </visual>
+      <collision>
+        <origin xyz="0 0 -0.026" rpy="0 0 0"/>
+        <geometry>
+          <mesh filename="package://iiwa_description/meshes/iiwa7/collision/link_5.stl"/>
+        </geometry>
+        <material name="Orange"/>
       </collision>
     </link>
@@ -224,30 +224,30 @@
       <axis xyz="0 0 1"/>
       <limit lower="${-120 * PI / 180}" upper="${120 * PI / 180}"
-	     effort="${max_effort}" velocity="${max_velocity}" />
+             effort="${max_effort}" velocity="${max_velocity}" />
       <safety_controller soft_lower_limit="${-118 * PI / 180}"
-			 soft_upper_limit="${118 * PI / 180}"
-			 k_position="${safety_controller_k_pos}"
-			 k_velocity="${safety_controller_k_vel}"/>
+                         soft_upper_limit="${118 * PI / 180}"
+                         k_position="${safety_controller_k_pos}"
+                         k_velocity="${safety_controller_k_vel}"/>
       <dynamics damping="${joint_damping}"/>
     </joint>
     <link name="${robot_name}_link_6">
       <inertial>
-	<origin xyz="0 0.0006 0.0004" rpy="0 0 0"/>
-	<mass value="2.3466"/>
-	<inertia ixx="0.006509"  ixy="0"  ixz="0" iyy="0.006259" iyz="0.00031891" izz="0.004527" />
-      </inertial>
-      <visual>
-	<origin xyz="0 0 0" rpy="0 0 0"/>
-	<geometry>
-	  <mesh filename="package://iiwa_description/meshes/iiwa7/visual/link_6.stl"/>
-	</geometry>
-	<material name="Orange"/>
-      </visual>
-      <collision>
-	<origin xyz="0 0 0" rpy="0 0 0"/>
-	<geometry>
-	  <mesh filename="package://iiwa_description/meshes/iiwa7/collision/link_6.stl"/>
-	</geometry>
-	<material name="Orange"/>
+        <origin xyz="0 0.0006 0.0004" rpy="0 0 0"/>
+        <mass value="2.3466"/>
+        <inertia ixx="0.006509"  ixy="0"  ixz="0" iyy="0.006259" iyz="0.00031891" izz="0.004527" />
+      </inertial>
+      <visual>
+        <origin xyz="0 0 0" rpy="0 0 0"/>
+        <geometry>
+          <mesh filename="package://iiwa_description/meshes/iiwa7/visual/link_6.stl"/>
+        </geometry>
+        <material name="Orange"/>
+      </visual>
+      <collision>
+        <origin xyz="0 0 0" rpy="0 0 0"/>
+        <geometry>
+          <mesh filename="package://iiwa_description/meshes/iiwa7/collision/link_6.stl"/>
+        </geometry>
+        <material name="Orange"/>
       </collision>
     </link>
@@ -258,30 +258,30 @@
       <axis xyz="0 0 1"/>
       <limit lower="${-175 * PI / 180}" upper="${175 * PI / 180}"
-	     effort="${max_effort}" velocity="${max_velocity}" />
+             effort="${max_effort}" velocity="${max_velocity}" />
       <safety_controller soft_lower_limit="${-173 * PI / 180}"
-			 soft_upper_limit="${173 * PI / 180}"
-			 k_position="${safety_controller_k_pos}"
-			 k_velocity="${safety_controller_k_vel}"/>
+                         soft_upper_limit="${173 * PI / 180}"
+                         k_position="${safety_controller_k_pos}"
+                         k_velocity="${safety_controller_k_vel}"/>
       <dynamics damping="${joint_damping}"/>
     </joint>
     <link name="${robot_name}_link_7">
       <inertial>
-	<origin xyz="0 0 0.02" rpy="0 0 0"/>
-	<mass value="3.129"/>
-	<inertia ixx="0.01464"  ixy="0.0005912"  ixz="0" iyy="0.01465" iyz="0" izz="0.002872" />
-      </inertial>
-      <visual>
-	<origin xyz="0 0 -0.0005" rpy="0 0 0"/>
-	<geometry>
-	  <mesh filename="package://iiwa_description/meshes/iiwa7/visual/link_7.stl"/>
-	</geometry>
-	<material name="Grey"/>
-      </visual>
-      <collision>
-	<origin xyz="0 0 -0.0005" rpy="0 0 0"/>
-	<geometry>
-	  <mesh filename="package://iiwa_description/meshes/iiwa7/collision/link_7.stl"/>
-	</geometry>
-	<material name="Grey"/>
+        <origin xyz="0 0 0.02" rpy="0 0 0"/>
+        <mass value="3.129"/>
+        <inertia ixx="0.01464"  ixy="0.0005912"  ixz="0" iyy="0.01465" iyz="0" izz="0.002872" />
+      </inertial>
+      <visual>
+        <origin xyz="0 0 -0.0005" rpy="0 0 0"/>
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
Commit message: fix URDF xacro files following the URDF conventions

File: iiwa_description/urdf/iiwa.transmission.xacro (robot description, xacro)
@@ -3,5 +3,4 @@
   <xacro:macro name="iiwa_transmission" params="hardware_interface">
     <transmission name="${robot_name}_tran_1">
-      <robotNamespace>/${robot_name}</robotNamespace>
       <type>transmission_interface/SimpleTransmission</type>
       <joint name="${robot_name}_joint_1">
@@ -9,10 +8,8 @@
       </joint>
       <actuator name="${robot_name}_motor_1">
-        <hardwareInterface>hardware_interface/${hardware_interface}</hardwareInterface>
         <mechanicalReduction>1</mechanicalReduction>
       </actuator>
     </transmission>
     <transmission name="${robot_name}_tran_2">
-      <robotNamespace>/${robot_name}</robotNamespace>
       <type>transmission_interface/SimpleTransmission</type>
       <joint name="${robot_name}_joint_2">
@@ -20,10 +17,8 @@
       </joint>
       <actuator name="${robot_name}_motor_2">
-        <hardwareInterface>hardware_interface/${hardware_interface}</hardwareInterface>
         <mechanicalReduction>1</mechanicalReduction>
       </actuator>
     </transmission>
     <transmission name="${robot_name}_tran_3">
-      <robotNamespace>/${robot_name}</robotNamespace>
       <type>transmission_interface/SimpleTransmission</type>
       <joint name="${robot_name}_joint_3">
@@ -31,10 +26,8 @@
       </joint>
       <actuator name="${robot_name}_motor_3">
-        <hardwareInterface>hardware_interface/${hardware_interface}</hardwareInterface>
         <mechanicalReduction>1</mechanicalReduction>
       </actuator>
     </transmission>
     <transmission name="${robot_name}_tran_4">
-      <robotNamespace>/${robot_name}</robotNamespace>
       <type>transmission_interface/SimpleTransmission</type>
       <joint name="${robot_name}_joint_4">
@@ -42,10 +35,8 @@
       </joint>
       <actuator name="${robot_name}_motor_4">
-        <hardwareInterface>hardware_interface/${hardware_interface}</hardwareInterface>
         <mechanicalReduction>1</mechanicalReduction>
       </actuator>
     </transmission>
     <transmission name="${robot_name}_tran_5">
-      <robotNamespace>/${robot_name}</robotNamespace>
       <type>transmission_interface/SimpleTransmission</type>
       <joint name="${robot_name}_joint_5">
@@ -53,10 +44,8 @@
       </joint>
       <actuator name="${robot_name}_motor_5">
-        <hardwareInterface>hardware_interface/${hardware_interface}</hardwareInterface>
         <mechanicalReduction>1</mechanicalReduction>
       </actuator>
     </transmission>
     <transmission name="${robot_name}_tran_6">
-      <robotNamespace>/${robot_name}</robotNamespace>
       <type>transmission_interface/SimpleTransmission</type>
       <joint name="${robot_name}_joint_6">
@@ -64,10 +53,8 @@
       </joint>
       <actuator name="${robot_name}_motor_6">
-        <hardwareInterface>hardware_interface/${hardware_interface}</hardwareInterface>
         <mechanicalReduction>1</mechanicalReduction>
       </actuator>
     </transmission>
     <transmission name="${robot_name}_tran_7">
-      <robotNamespace>/${robot_name}</robotNamespace>
       <type>transmission_interface/SimpleTransmission</type>
       <joint name="${robot_name}_joint_7">
@@ -75,5 +62,4 @@
       </joint>
       <actuator name="${robot_name}_motor_7">
-        <hardwareInterface>hardware_interface/${hardware_interface}</hardwareInterface>
         <mechanicalReduction>1</mechanicalReduction>
       </actuator>

File: iiwa_description/urdf/iiwa14.xacro (robot description, xacro)
@@ -38,12 +38,11 @@
           <mesh filename="package://iiwa_description/meshes/iiwa14/collision/link_0.stl"/>
         </geometry>
-        <material name="Grey"/>
-      </collision>
-      <self_collision_checking>
+      </collision>
+      <!-- <self_collision_checking>
         <origin xyz="0 0 0" rpy="0 0 0"/>
         <geometry>
           <capsule radius="0.15" length="0.25"/>
         </geometry>
-      </self_collision_checking>
+      </self_collision_checking> -->
     </link>
     <!-- joint between link_0 and link_1 -->
@@ -79,5 +78,4 @@
           <mesh filename="package://iiwa_description/meshes/iiwa14/collision/link_1.stl"/>
         </geometry>
-        <material name="Orange"/>
       </collision>
     </link>
@@ -114,5 +112,4 @@
           <mesh filename="package://iiwa_description/meshes/iiwa14/collision/link_2.stl"/>
         </geometry>
-        <material name="Orange"/>
       </collision>
     </link>
@@ -149,5 +146,4 @@
           <mesh filename="package://iiwa_description/meshes/iiwa14/collision/link_3.stl"/>
         </geometry>
-        <material name="Orange"/>
       </collision>
     </link>
@@ -184,5 +180,4 @@
           <mesh filename="package://iiwa_description/meshes/iiwa14/collision/link_4.stl"/>
         </geometry>
-        <material name="Orange"/>
       </collision>
     </link>
@@ -219,5 +214,4 @@
           <mesh filename="package://iiwa_description/meshes/iiwa14/collision/link_5.stl"/>
         </geometry>
-        <material name="Orange"/>
       </collision>
     </link>
@@ -254,5 +248,4 @@
           <mesh filename="package://iiwa_description/meshes/iiwa14/collision/link_6.stl"/>
         </geometry>
-        <material name="Orange"/>
       </collision>
     </link>
@@ -289,5 +282,4 @@
           <mesh filename="package://iiwa_description/meshes/iiwa14/collision/link_7.stl"/>
         </geometry>
-        <material name="Grey"/>
       </collision>
     </link>

File: iiwa_description/urdf/iiwa7.xacro (robot description, xacro)
@@ -38,12 +38,11 @@
           <mesh filename="package://iiwa_description/meshes/iiwa7/collision/link_0.stl"/>
         </geometry>
-        <material name="Grey"/>
-      </collision>
-      <self_collision_checking>
+      </collision>
+      <!-- <self_collision_checking>
         <origin xyz="0 0 0" rpy="0 0 0"/>
         <geometry>
           <capsule radius="0.15" length="0.25"/>
         </geometry>
-      </self_collision_checking>
+      </self_collision_checking> -->
     </link>
     <!-- joint between link_0 and link_1 -->
@@ -79,5 +78,4 @@
           <mesh filename="package://iiwa_description/meshes/iiwa7/collision/link_1.stl"/>
         </geometry>
-        <material name="Orange"/>
       </collision>
     </link>
@@ -113,5 +111,4 @@
           <mesh filename="package://iiwa_description/meshes/iiwa7/collision/link_2.stl"/>
         </geometry>
-        <material name="Orange"/>
       </collision>
     </link>
@@ -147,5 +144,4 @@
           <mesh filename="package://iiwa_description/meshes/iiwa7/collision/link_3.stl"/>
         </geometry>
-        <material name="Orange"/>
       </collision>
     </link>
@@ -181,5 +177,4 @@
           <mesh filename="package://iiwa_description/meshes/iiwa7/collision/link_4.stl"/>
         </geometry>
-        <material name="Orange"/>
       </collision>
     </link>
@@ -215,5 +210,4 @@
           <mesh filename="package://iiwa_description/meshes/iiwa7/collision/link_5.stl"/>
         </geometry>
-        <material name="Orange"/>
       </collision>
     </link>
@@ -249,5 +243,4 @@
           <mesh filename="package://iiwa_description/meshes/iiwa7/collision/link_6.stl"/>
         </geometry>
-        <material name="Orange"/>
       </collision>
     </link>
@@ -283,5 +276,4 @@
           <mesh filename="package://iiwa_description/meshes/iiwa7/collision/link_7.stl"/>
         </geometry>
-        <material name="Grey"/>
       </collision>
     </link>
